Commit message: Single robot Spawn and control

File: descriptions/urdf/volta/components/wheel_volta.urdf.xacro (robot description, xacro)
@@ -28,5 +28,5 @@
     <xacro:macro name="volta_wheel" params="wheel_prefix *joint_origin">
         <!-- Wheel Link -->
-        <link name="${wheel_prefix}_wheel_${number}">
+        <link name="${wheel_prefix}_wheel">
             <visual>
                 <origin xyz="0 0 0" rpy="1.570796327 0 0"/>
@@ -48,5 +48,5 @@
             </inertial>
         </link>
-        <gazebo reference="${wheel_prefix}_wheel_${number}">
+        <gazebo reference="${wheel_prefix}_wheel">
             <material>Gazebo/Red</material>
             <mu1 value="1400"/>
@@ -57,14 +57,14 @@
         </gazebo>
         <!-- Wheel Joint -->
-        <joint name="${wheel_prefix}_wheel_${number}_joint_${number}" type="continuous">
+        <joint name="${wheel_prefix}_wheel_joint" type="continuous">
             <parent link="base_link_${number}"/>
-            <child link="${wheel_prefix}_wheel_${number}" />
+            <child link="${wheel_prefix}_wheel" />
             <xacro:insert_block name="joint_origin" />
             <axis xyz="0 1 0" />
         </joint>
         <!-- Wheel Transmission -->
-        <transmission name="${wheel_prefix}_wheel_${number}_transmission" type="SimpleTransmission">
+        <transmission name="${wheel_prefix}_wheel_transmission" type="SimpleTransmission">
             <type>transmission_interface/SimpleTransmission</type>
-            <joint name="${wheel_prefix}_wheel_${number}_joint_${number}">
+            <joint name="${wheel_prefix}_wheel_joint">
                 <hardwareInterface>hardware_interface/VelocityJointInterface</hardwareInterface>
             </joint>

File: descriptions/urdf/volta/volta.urdf.xacro (robot description, xacro)
@@ -77,8 +77,8 @@
         </link>
         <!-- Wheel -->
-        <xacro:volta_wheel wheel_prefix="right_${number}">
+        <xacro:volta_wheel wheel_prefix="right">
             <origin xyz="0.0 ${-wheel_joint_y_abs} ${wheel_joint_z_abs}" rpy="0 0 0" />
         </xacro:volta_wheel>
-        <xacro:volta_wheel wheel_prefix="left_${number}">
+        <xacro:volta_wheel wheel_prefix="left">
             <origin xyz="0.0 ${wheel_joint_y_abs} ${wheel_joint_z_abs}" rpy="0 0 0" />
         </xacro:volta_wheel>
@@ -114,4 +114,5 @@
         <gazebo>
             <plugin name="gazebo_ros_control" filename="libgazebo_ros_control.so">
+                <!-- <robotParam>/volta${number}/robot_description</robotParam> -->
                 <robotNamespace>$(arg robot_namespace)</robotNamespace>
                 <robotSimType>gazebo_ros_control/DefaultRobotHWSim</robotSimType>

File: descriptions/urdf/volta/volta.xacro (robot description, xacro)
@@ -26,5 +26,4 @@
   <xacro:arg name="number" default="0" />
   <xacro:include filename="$(find descriptions)/urdf/volta/volta.urdf.xacro" />
-  <!-- <xacro:volta number="0"></xacro:volta> -->
   <xacro:volta_robot number="$(arg number)"/>
 </robot>
