Commit message: Setting up for third volta (second follower)

File: descriptions/urdf/volta0/accessories/lidar_volta.urdf.xacro (robot description, xacro)
@@ -26,5 +26,5 @@
 <robot name="volta_robot_0" xmlns:xacro="https://ros.org/wiki/xacro">
   <xacro:macro name="lidar" params="frame:=lidar topic:=scan_filtered sample_size:=271 update_rate:=50
-                 min_angle:=-1.57 max_angle:=1.57 min_range:=0.5 max_range:=10.0 rplidar_a3_enabled:=true hokuyo_ust_10lx_enabled:=false robot_namespace:=/">
+                 min_angle:=-3.14159 max_angle:=3.14159 min_range:=0.5 max_range:=10.0 rplidar_a3_enabled:=true hokuyo_ust_10lx_enabled:=false robot_namespace:=/">
       <xacro:if value="${rplidar_a3_enabled}">
         <!-- RPLidar mount x position -->

File: descriptions/urdf/volta2/accessories/camera_volta.urdf.xacro (robot description, xacro)
@@ -24,5 +24,5 @@
 SOFTWARE, EVEN IF ADVISED OF THE POSSIBILITY OF SUCH DAMAGE.
 -->
-<robot name="volta_robot_0" xmlns:xacro="https://ros.org/wiki/xacro">
+<robot name="volta" xmlns:xacro="https://ros.org/wiki/xacro">
     <xacro:macro name="camera_" params="frame:=camera topic:=camera info_topic:=camera_info update_rate:=50 intel_d435i_enabled:=true orbbec_astra_pro_enabled:=false robot_namespace:=/">
         <xacro:if value="${intel_d435i_enabled}">

File: descriptions/urdf/volta2/accessories/imu_volta.urdf.xacro (robot description, xacro)
@@ -24,5 +24,5 @@
 SOFTWARE, EVEN IF ADVISED OF THE POSSIBILITY OF SUCH DAMAGE.
 -->
-<robot name="volta_robot_0" xmlns:xacro="https://ros.org/wiki/xacro">
+<robot name="volta_robot_2" xmlns:xacro="https://ros.org/wiki/xacro">
     <xacro:macro name="imu" params="frame:=imu topic:=imu/data update_rate:=50 robot_namespace:=/ tf_pre:=/">
         <joint name="${frame}_joint" type="fixed">

File: descriptions/urdf/volta2/accessories/lidar_volta.urdf.xacro (robot description, xacro)
@@ -24,5 +24,5 @@
 SOFTWARE, EVEN IF ADVISED OF THE POSSIBILITY OF SUCH DAMAGE.
 -->
-<robot name="volta_robot_1" xmlns:xacro="https://ros.org/wiki/xacro">
+<robot name="volta_robot_2" xmlns:xacro="https://ros.org/wiki/xacro">
   <xacro:macro name="lidar" params="frame:=lidar topic:=scan_filtered sample_size:=271 update_rate:=50
                  min_angle:=-3.14159 max_angle:=3.14159 min_range:=0.5 max_range:=10.0 rplidar_a3_enabled:=true hokuyo_ust_10lx_enabled:=false robot_namespace:=/">
@@ -111,6 +111,6 @@
           </ray>
           <plugin name="gazebo_ros_laser" filename="libgazebo_ros_laser.so">
-            <topicName>volta_1/${topic}</topicName>
-            <frameName>volta_1_tf/${frame}</frameName>
+            <topicName>volta_2/${topic}</topicName>
+            <frameName>volta_2_tf/${frame}</frameName>
             <robotNamespace>${robot_namespace}</robotNamespace>
             <gaussianNoise>0.005</gaussianNoise>

File: descriptions/urdf/volta2/components/caster_volta.urdf.xacro (robot description, xacro)
@@ -24,32 +24,41 @@
 SOFTWARE, EVEN IF ADVISED OF THE POSSIBILITY OF SUCH DAMAGE.
 -->
-<robot name="volta_robot_0" xmlns:xacro="https://ros.org/wiki/xacro">
-    <xacro:macro name="imu" params="frame:=imu topic:=imu/data update_rate:=50 robot_namespace:=/ tf_pre:=/">
-        <joint name="${frame}_joint" type="fixed">
-            <parent link="base_link" />
-            <child link="${frame}" />
-            <origin xyz="0 0 ${base_h/2}" rpy="0 0 0" />
-        </joint>
-        <link name="${frame}">
+<robot name="volta_robot_2" xmlns:xacro="https://ros.org/wiki/xacro">
+    <!-- Caster Macro -->
+    <xacro:macro name="volta_caster" params="caster_prefix *caster_joint_origin">
+        <!-- Caster Joint -->
+        <link name="caster_${caster_prefix}_link">
+            <visual>
+                <origin rpy="0 0 0" xyz="0.0 0.0 0.0"/>
+                <geometry>
+                    <sphere radius="${caster_radius}"/>
+                </geometry>
+                <material name="black"/>
+            </visual>
+            <collision>
+                <geometry>
+                    <sphere radius="${caster_radius}"/>
+                </geometry>
+                <origin rpy="0 0 0" xyz="0 0 0"/>
+            </collision>
             <inertial>
-                <mass value="0.001"/>
-                <origin xyz="0 0 0" rpy="0 0 0"/>
-                <inertia ixx="1e-09" ixy="0.0" ixz="0.0" iyy="1e-09" iyz="0.0" izz="1e-09"/>
+                <mass value="0.1"/>
+                <origin xyz="0 0 0"/>
+                <inertia ixx="0.0001" ixy="0.0" ixz="0.0" iyy="0.0001" iyz="0.0" izz="0.0001"/>
             </inertial>
         </link>
-        <gazebo>
-            <plugin name="imu_plugin" filename="libgazebo_ros_imu.so">
-                <alwaysOn>true</alwaysOn>
-                <robotNamespace>${robot_namespace}</robotNamespace>
-                <updateRate>${update_rate}</updateRate>
-                <bodyName>${frame}</bodyName>
-                <frameId>${tf_pre}${frame}</frameId>
-                <frameName>${tf_pre}${frame}</frameName>
-                <topicName>${topic}</topicName>
-                <xyzOffset>0.0 0.0 0.0</xyzOffset>
-                <rpyOffset>0.0 0.0 0.0</rpyOffset>
-                <headingDrift>0.0005</headingDrift>
-                <gaussianNoise>0.0005</gaussianNoise>
-            </plugin>
+        <!-- Caster Joint -->
+        <joint name="caster_${caster_prefix}_joint" type="fixed">
+            <parent link="base_link"/>
+            <child link="caster_${caster_prefix}_link"/>
+            <xacro:insert_block name="caster_joint_origin" />
+        </joint>
+        <gazebo reference="caster_${caster_prefix}_link">
+            <material>Gazebo/DarkGrey</material>
+            <turnGravityOff>false</turnGravityOff>
+            <mu1 value="0.1"/>
+            <mu2 value="0.1"/>
+            <kp value="10000000.0"></kp>
+            <kd value="1.0"></kd>
         </gazebo>
     </xacro:macro>

File: descriptions/urdf/volta2/volta.xacro (robot description, xacro)
@@ -1,3 +1,2 @@
-<?xml version="1.0"?>
 <!--
 Copyright (c) 2020, Botsync Pte. Ltd.
@@ -24,33 +23,6 @@
 SOFTWARE, EVEN IF ADVISED OF THE POSSIBILITY OF SUCH DAMAGE.
 -->
-<robot name="volta_robot_0" xmlns:xacro="https://ros.org/wiki/xacro">
-    <xacro:macro name="imu" params="frame:=imu topic:=imu/data update_rate:=50 robot_namespace:=/ tf_pre:=/">
-        <joint name="${frame}_joint" type="fixed">
-            <parent link="base_link" />
-            <child link="${frame}" />
-            <origin xyz="0 0 ${base_h/2}" rpy="0 0 0" />
-        </joint>
-        <link name="${frame}">
-            <inertial>
-                <mass value="0.001"/>
-                <origin xyz="0 0 0" rpy="0 0 0"/>
-                <inertia ixx="1e-09" ixy="0.0" ixz="0.0" iyy="1e-09" iyz="0.0" izz="1e-09"/>
-            </inertial>
-        </link>
-        <gazebo>
-            <plugin name="imu_plugin" filename="libgazebo_ros_imu.so">
-                <alwaysOn>true</alwaysOn>
-                <robotNamespace>${robot_namespace}</robotNamespace>
-                <updateRate>${update_rate}</updateRate>
-                <bodyName>${frame}</bodyName>
-                <frameId>${tf_pre}${frame}</frameId>
-                <frameName>${tf_pre}${frame}</frameName>
-                <topicName>${topic}</topicName>
-                <xyzOffset>0.0 0.0 0.0</xyzOffset>
-                <rpyOffset>0.0 0.0 0.0</rpyOffset>
-                <headingDrift>0.0005</headingDrift>
-                <gaussianNoise>0.0005</gaussianNoise>
-            </plugin>
-        </gazebo>
-    </xacro:macro>
+<robot name="volta_robot_2" xmlns:xacro="https://ros.org/wiki/xacro">
+  <xacro:include filename="$(find descriptions)/urdf/volta2/volta.urdf.xacro" />
+  <xacro:volta_robot_2/>
 </robot>
