Commit message: Simple leader follower working

File: descriptions/urdf/volta/accessories/camera_volta.urdf.xacro (robot description, xacro)
@@ -25,5 +25,5 @@
 -->
 <robot name="volta" xmlns:xacro="https://ros.org/wiki/xacro">
-    <xacro:macro name="camera_" params="frame:=camera_${number} topic:=camera info_topic:=camera_info update_rate:=50 intel_d435i_enabled:=true orbbec_astra_pro_enabled:=false robot_namespace:=/">
+    <xacro:macro name="camera_" params="frame:=camera topic:=camera info_topic:=camera_info update_rate:=50 intel_d435i_enabled:=true orbbec_astra_pro_enabled:=false robot_namespace:=/">
         <xacro:if value="${intel_d435i_enabled}">
           <!-- Camera link -->
@@ -49,5 +49,5 @@
           <!-- Camera joint -->
           <joint name="base_to_camera" type="fixed">
-              <parent link="base_link_${number}"/>
+              <parent link="base_link"/>
               <child link="${frame}"/>
               <origin xyz="${camera_joint_x} ${camera_joint_y} ${camera_joint_z + 0.0125}"/>
@@ -77,5 +77,5 @@
           <!-- Camera joint -->
           <joint name="base_to_camera" type="fixed">
-              <parent link="base_link_${number}"/>
+              <parent link="base_link"/>
               <child link="${frame}"/>
               <origin xyz="${camera_joint_x} ${camera_joint_y} ${camera_joint_z + 0.0337}"/>

File: descriptions/urdf/volta/accessories/imu_volta.urdf.xacro (robot description, xacro)
@@ -26,10 +26,10 @@
 <robot name="volta" xmlns:xacro="https://ros.org/wiki/xacro">
     <xacro:macro name="imu" params="frame:=imu topic:=imu/data update_rate:=50 robot_namespace:=/ tf_pre:=/">
-        <joint name="${frame}_${number}_joint_${number}" type="fixed">
-            <parent link="base_link_${number}" />
-            <child link="${frame}_${number}" />
+        <joint name="${frame}_joint" type="fixed">
+            <parent link="base_link" />
+            <child link="${frame}" />
             <origin xyz="0 0 ${base_h/2}" rpy="0 0 0" />
         </joint>
-        <link name="${frame}_${number}">
+        <link name="${frame}">
             <inertial>
                 <mass value="0.001"/>
@@ -43,7 +43,7 @@
                 <robotNamespace>${robot_namespace}</robotNamespace>
                 <updateRate>${update_rate}</updateRate>
-                <bodyName>${frame}_${number}</bodyName>
-                <frameId>${tf_pre}${frame}_${number}</frameId>
-                <frameName>${tf_pre}${frame}_${number}</frameName>
+                <bodyName>${frame}</bodyName>
+                <frameId>${tf_pre}${frame}</frameId>
+                <frameName>${tf_pre}${frame}</frameName>
                 <topicName>${topic}</topicName>
                 <xyzOffset>0.0 0.0 0.0</xyzOffset>

File: descriptions/urdf/volta/accessories/lidar_volta.urdf.xacro (robot description, xacro)
@@ -25,5 +25,5 @@
 -->
 <robot name="volta" xmlns:xacro="https://ros.org/wiki/xacro">
-  <xacro:macro name="lidar" params="frame:=lidar_${number} topic:=scan_filtered sample_size:=271 update_rate:=50
+  <xacro:macro name="lidar" params="frame:=lidar topic:=scan_filtered sample_size:=271 update_rate:=50
                  min_angle:=-1.57 max_angle:=1.57 min_range:=0.5 max_range:=10.0 rplidar_a3_enabled:=true hokuyo_ust_10lx_enabled:=false robot_namespace:=/">
       <xacro:if value="${rplidar_a3_enabled}">
@@ -53,5 +53,5 @@
         <joint name="lidar_joint" type="fixed">
             <origin xyz="${lidar_joint_x} ${lidar_joint_y} ${lidar_joint_z + 0.03}" rpy="0 0 0" />
-            <parent link="base_link_${number}" />
+            <parent link="base_link" />
             <child link="${frame}" />
         </joint>
@@ -85,5 +85,5 @@
         <joint name="lidar_joint" type="fixed">
             <origin xyz="${lidar_joint_x} ${lidar_joint_y} ${lidar_joint_z + 0.049}" rpy="0 0 0" />
-            <parent link="base_link_${number}" />
+            <parent link="base_link" />
             <child link="${frame}" />
         </joint>

File: descriptions/urdf/volta/components/caster_volta.urdf.xacro (robot description, xacro)
@@ -28,5 +28,5 @@
     <xacro:macro name="volta_caster" params="caster_prefix *caster_joint_origin">
         <!-- Caster Joint -->
-        <link name="caster_${caster_prefix}_link_${number}">
+        <link name="caster_${caster_prefix}_link">
             <visual>
                 <origin rpy="0 0 0" xyz="0.0 0.0 0.0"/>
@@ -34,5 +34,5 @@
                     <sphere radius="${caster_radius}"/>
                 </geometry>
-                <material name="Black"/>
+                <material name="black"/>
             </visual>
             <collision>
@@ -49,10 +49,10 @@
         </link>
         <!-- Caster Joint -->
-        <joint name="caster_${caster_prefix}_joint_${number}" type="fixed">
-            <parent link="base_link_${number}"/>
-            <child link="caster_${caster_prefix}_link_${number}"/>
+        <joint name="caster_${caster_prefix}_joint" type="fixed">
+            <parent link="base_link"/>
+            <child link="caster_${caster_prefix}_link"/>
             <xacro:insert_block name="caster_joint_origin" />
         </joint>
-        <gazebo reference="caster_${caster_prefix}_link_${number}">
+        <gazebo reference="caster_${caster_prefix}_link">
             <material>Gazebo/DarkGrey</material>
             <turnGravityOff>false</turnGravityOff>

File: descriptions/urdf/volta/components/wheel_volta.urdf.xacro (robot description, xacro)
@@ -58,5 +58,5 @@
         <!-- Wheel Joint -->
         <joint name="${wheel_prefix}_wheel_joint" type="continuous">
-            <parent link="base_link_${number}"/>
+            <parent link="base_link"/>
             <child link="${wheel_prefix}_wheel" />
             <xacro:insert_block name="joint_origin" />

File: descriptions/urdf/volta/volta.urdf.xacro (robot description, xacro)
@@ -25,5 +25,4 @@
 -->
 <robot name="volta_robot" xmlns:xacro="https://ros.org/wiki/xacro">
-    <xacro:macro name="volta_robot" params="number:=0">
     <!-- xacro includes -->
     <xacro:include filename="$(find descriptions)/urdf/volta/volta_properties.xacro"/>
@@ -35,22 +34,23 @@
     <xacro:arg name="robot_namespace" default="/" />
     <xacro:arg name="tf_pre" default=""/>
-    <xacro:arg name="lidar_enabled" default="true"/>
-    <xacro:arg name="rplidar_a3_enabled" default="true"/>
+    <xacro:arg name="lidar_enabled" default="false"/>
+    <xacro:arg name="rplidar_a3_enabled" default="false"/>
     <xacro:arg name="hokuyo_ust_10lx_enabled" default="false"/>
-    <xacro:arg name="imu_enabled" default="true"/>
-    <xacro:arg name="camera_enabled" default="true"/>
-    <xacro:arg name="intel_d435i_enabled" default="true"/>
+    <xacro:arg name="imu_enabled" default="false"/>
+    <xacro:arg name="camera_enabled" default="false"/>
+    <xacro:arg name="intel_d435i_enabled" default="false"/>
     <xacro:arg name="orbbec_astra_pro_enabled" default="false"/>
-        <!-- Footprint_${number} -->
-        <link name="footprint_${number}"/>
-        <!-- Joint from footprint_${number} to base link(chassis) -->
-        <joint name="base_footprint_${number}_joint" type="fixed">
+    <xacro:macro name="volta_robot">
+        <!-- Footprint -->
+        <link name="footprint"/>
+        <!-- Joint from footprint to base link(chassis) -->
+        <joint name="base_footprint_joint" type="fixed">
             <origin xyz="0 0 ${base_underside_h}" rpy="0 0 0" />
-            <parent link="base_link_${number}" />
-            <child link="footprint_${number}" />
+            <parent link="base_link" />
+            <child link="footprint" />
         </joint>
-        <!-- Chassis a.k.a base_link_${number} -->
-        <link name="base_link_${number}">
-            <visual name="visual_base_${number}">
+        <!-- Chassis a.k.a base_link -->
+        <link name="base_link">
+            <visual name="visual_base">
                 <origin xyz="0 0 0" rpy="0 0 0" />
                 <geometry>
@@ -58,5 +58,5 @@
                 </geometry>
             </visual>
-            <visual name="visual_logo_${number}">
+            <visual name="visual_logo">
                 <origin xyz="0 0 0" rpy="0 0 0" />
                 <geometry>
@@ -84,14 +84,14 @@
         </xacro:volta_wheel>
         <!-- Caster wheels -->
-        <xacro:volta_caster caster_prefix="front_left_${number}">
+        <xacro:volta_caster caster_prefix="front_left">
             <origin xyz="${caster_joint_x} ${caster_joint_y} ${caster_joint_z}" rpy="0 0 0" />
         </xacro:volta_caster>
-        <xacro:volta_caster caster_prefix="front_right_${number}">
+        <xacro:volta_caster caster_prefix="front_right">
             <origin xyz="${caster_joint_x} ${-caster_joint_y} ${caster_joint_z}" rpy="0 0 0" />
         </xacro:volta_caster>
-        <xacro:volta_caster caster_prefix="rear_right_${number}">
+        <xacro:volta_caster caster_prefix="rear_right">
             <origin xyz="${-caster_joint_x} ${-caster_joint_y} ${caster_joint_z}" rpy="0 0 0" />
         </xacro:volta_caster>
-        <xacro:volta_caster caster_prefix="rear_left_${number}">
+        <xacro:volta_caster caster_prefix="rear_left">
             <origin xyz="${-caster_joint_x} ${caster_joint_y} ${caster_joint_z}" rpy="0 0 0" />
         </xacro:volta_caster>
@@ -114,5 +114,4 @@
         <gazebo>
             <plugin name="gazebo_ros_control" filename="libgazebo_ros_control.so">
-                <!-- <robotParam>/volta${number}/robot_description</robotParam> -->
                 <robotNamespace>$(arg robot_namespace)</robotNamespace>
                 <robotSimType>gazebo_ros_control/DefaultRobotHWSim</robotSimType>
@@ -120,4 +119,3 @@
         </gazebo>
     </xacro:macro>
-<!-- </xacro:macro> -->
 </robot>

File: descriptions/urdf/volta/volta.xacro (robot description, xacro)
@@ -24,6 +24,5 @@
 -->
 <robot name="volta_robot" xmlns:xacro="https://ros.org/wiki/xacro">
-  <xacro:arg name="number" default="0" />
   <xacro:include filename="$(find descriptions)/urdf/volta/volta.urdf.xacro" />
-  <xacro:volta_robot number="$(arg number)"/>
+  <xacro:volta_robot/>
 </robot>

File: descriptions/urdf/volta0/accessories/camera_volta.urdf.xacro (robot description, xacro)
@@ -32,5 +32,5 @@
                   <origin xyz="0 0 -0.0125" rpy="0 0 0"/>
                   <geometry>
-                      <mesh filename="package://volta_description/meshes/d435i.dae"/>
+                      <mesh filename="package://descriptions/meshes/d435i.dae"/>
                   </geometry>
               </visual>
@@ -38,5 +38,5 @@
                   <origin xyz="0 0 -0.0125" rpy="0 0 0"/>
                   <geometry>
-                      <mesh filename="package://volta_description/meshes/d435i.dae"/>
+                      <mesh filename="package://descriptions/meshes/d435i.dae"/>
                   </geometry>
               </collision>
@@ -60,5 +60,5 @@
                   <origin xyz="0 0 -0.0337" rpy="0 0 0"/>
                   <geometry>
-                      <mesh filename="package://volta_description/meshes/astra.dae"/>
+                      <mesh filename="package://descriptions/meshes/astra.dae"/>
                   </geometry>
               </visual>
@@ -66,5 +66,5 @@
                   <origin xyz="0 0 -0.0337" rpy="0 0 0"/>
                   <geometry>
-                      <mesh filename="package://volta_description/meshes/astra.dae"/>
+                      <mesh filename="package://descriptions/meshes/astra.dae"/>
                   </geometry>
               </collision>

File: descriptions/urdf/volta0/accessories/lidar_volta.urdf.xacro (robot description, xacro)
@@ -35,5 +35,5 @@
                 <origin xyz="0 0 -0.03" rpy="0 0 0.785398"/>
                 <geometry>
-                    <mesh filename="package://volta_description/meshes/rplidar.dae"/>
+                    <mesh filename="package://descriptions/meshes/rplidar.dae"/>
                 </geometry>
             </visual>
@@ -41,5 +41,5 @@
                 <origin xyz="0 0 -0.03" rpy="0 0 0"/>
                 <geometry>
-                  <mesh filename="package://volta_description/meshes/rplidar.dae"/>
+                  <mesh filename="package://descriptions/meshes/rplidar.dae"/>
                 </geometry>
             </collision>
@@ -67,5 +67,5 @@
               <origin xyz="0 0 -0.049" rpy="0 0 0"/>
                 <geometry>
-                    <mesh filename="package://volta_description/meshes/hokuyo.dae"/>
+                    <mesh filename="package://descriptions/meshes/hokuyo.dae"/>
                 </geometry>
             </visual>
@@ -73,5 +73,5 @@
                 <origin xyz="0 0 -0.049" rpy="0 0 0"/>
                 <geometry>
-                  <mesh filename="package://volta_description/meshes/hokuyo.dae"/>
+                  <mesh filename="package://descriptions/meshes/hokuyo.dae"/>
                 </geometry>
             </collision>

File: descriptions/urdf/volta0/components/caster_volta.urdf.xacro (robot description, xacro)
@@ -24,5 +24,5 @@
 SOFTWARE, EVEN IF ADVISED OF THE POSSIBILITY OF SUCH DAMAGE.
 -->
-<robot name="volta_robot" xmlns:xacro="https://ros.org/wiki/xacro">
+<robot name="volta_robot_0" xmlns:xacro="https://ros.org/wiki/xacro">
     <!-- Caster Macro -->
     <xacro:macro name="volta_caster" params="caster_prefix *caster_joint_origin">
@@ -34,5 +34,5 @@
                     <sphere radius="${caster_radius}"/>
                 </geometry>
-                <material name="Black"/>
+                <material name="black"/>
             </visual>
             <collision>

File: descriptions/urdf/volta0/components/wheel_volta.urdf.xacro (robot description, xacro)
@@ -24,5 +24,5 @@
 SOFTWARE, EVEN IF ADVISED OF THE POSSIBILITY OF SUCH DAMAGE.
 -->
-<robot name="volta_robot" xmlns:xacro="https://ros.org/wiki/xacro">
+<robot name="volta_robot_0" xmlns:xacro="https://ros.org/wiki/xacro">
     <!-- Wheel Macro -->
     <xacro:macro name="volta_wheel" params="wheel_prefix *joint_origin">

File: descriptions/urdf/volta0/volta.urdf.xacro (robot description, xacro)
@@ -24,9 +24,9 @@
 SOFTWARE, EVEN IF ADVISED OF THE POSSIBILITY OF SUCH DAMAGE.
 -->
-<robot name="volta_robot" xmlns:xacro="https://ros.org/wiki/xacro">
+<robot name="volta_robot_0" xmlns:xacro="https://ros.org/wiki/xacro">
     <!-- xacro includes -->
-    <xacro:include filename="$(find volta_description)/urdf/volta_properties.xacro"/>
-    <xacro:include filename="$(find volta_description)/urdf/components/wheel_volta.urdf.xacro"/>
-    <xacro:include filename="$(find volta_description)/urdf/components/caster_volta.urdf.xacro"/>
+    <xacro:include filename="$(find descriptions)/urdf/volta0/volta_properties.xacro"/>
+    <xacro:include filename="$(find descriptions)/urdf/volta0/components/wheel_volta.urdf.xacro"/>
+    <xacro:include filename="$(find descriptions)/urdf/volta0/components/caster_volta.urdf.xacro"/>
     <!-- xacro properties -->
     <xacro:property name="PI" value="3.14159"/>
@@ -34,12 +34,12 @@
     <xacro:arg name="robot_namespace" default="/" />
     <xacro:arg name="tf_pre" default=""/>
-    <xacro:arg name="lidar_enabled" default="true"/>
-    <xacro:arg name="rplidar_a3_enabled" default="true"/>
+    <xacro:arg name="lidar_enabled" default="false"/>
+    <xacro:arg name="rplidar_a3_enabled" default="false"/>
     <xacro:arg name="hokuyo_ust_10lx_enabled" default="false"/>
-    <xacro:arg name="imu_enabled" default="true"/>
-    <xacro:arg name="camera_enabled" default="true"/>
-    <xacro:arg name="intel_d435i_enabled" default="true"/>
+    <xacro:arg name="imu_enabled" default="false"/>
+    <xacro:arg name="camera_enabled" default="false"/>
+    <xacro:arg name="intel_d435i_enabled" default="false"/>
     <xacro:arg name="orbbec_astra_pro_enabled" default="false"/>
-    <xacro:macro name="volta_robot">
+    <xacro:macro name="volta_robot_0">
         <!-- Footprint -->
         <link name="footprint"/>
@@ -55,5 +55,5 @@
                 <origin xyz="0 0 0" rpy="0 0 0" />
                 <geometry>
-                    <mesh filename="package://volta_description/meshes/volta.dae"/>
+                    <mesh filename="package://descriptions/meshes/volta.dae"/>
                 </geometry>
             </visual>
@@ -61,5 +61,5 @@
                 <origin xyz="0 0 0" rpy="0 0 0" />
                 <geometry>
-                    <mesh filename="package://volta_description/meshes/volta_logo.dae"/>
+                    <mesh filename="package://descriptions/meshes/volta_logo.dae"/>
                 </geometry>
             </visual>
@@ -67,5 +67,5 @@
                 <origin xyz="0 0 0" rpy="0 0 0" />
                 <geometry>
-                    <mesh filename="package://volta_description/meshes/volta.dae"/>
+                    <mesh filename="package://descriptions/meshes/volta.dae"/>
                 </geometry>
             </collision>
@@ -98,24 +98,44 @@
         <!-- IMU -->
         <xacro:if value="$(arg imu_enabled)">
-            <xacro:include filename="$(find volta_description)/urdf/accessories/imu_volta.urdf.xacro"/>
+            <xacro:include filename="$(find descriptions)/urdf/volta0/accessories/imu_volta.urdf.xacro"/>
             <xacro:imu robot_namespace="$(arg robot_namespace)" tf_pre="$(arg tf_pre)"></xacro:imu>
         </xacro:if>
         <!-- LIDAR -->
         <xacro:if value="$(arg lidar_enabled)">
-            <xacro:include filename="$(find volta_description)/urdf/accessories/lidar_volta.urdf.xacro"/>
+            <xacro:include filename="$(find descriptions)/urdf/volta0/accessories/lidar_volta.urdf.xacro"/>
             <xacro:lidar rplidar_a3_enabled="$(arg rplidar_a3_enabled)" hokuyo_ust_10lx_enabled="$(arg hokuyo_ust_10lx_enabled)" robot_namespace="$(arg robot_namespace)">  </xacro:lidar>
         </xacro:if>
         <!-- Camera -->
         <xacro:if value="$(arg camera_enabled)">
-            <xacro:include filename="$(find volta_description)/urdf/accessories/camera_volta.urdf.xacro"/>
+            <xacro:include filename="$(find descriptions)/urdf/volta0/accessories/camera_volta.urdf.xacro"/>
             <xacro:camera_ intel_d435i_enabled="$(arg intel_d435i_enabled)" orbbec_astra_pro_enabled="$(arg orbbec_astra_pro_enabled)" robot_namespace="$(arg robot_namespace)"></xacro:camera_>
         </xacro:if>
         <!-- Robot Gazebo tag -->
-        <gazebo>
+        <!-- <gazebo>
             <plugin name="gazebo_ros_control" filename="libgazebo_ros_control.so">
                 <robotNamespace>$(arg robot_namespace)</robotNamespace>
                 <robotSimType>gazebo_ros_control/DefaultRobotHWSim</robotSimType>
             </plugin>
-        </gazebo>
+        </gazebo> -->
+        <gazebo>
+            <plugin name="differential_drive_controller" filename="libgazebo_ros_diff_drive.so">
+                <updateRate>20</updateRate>
+                <leftJoint>left_wheel_joint</leftJoint>
+                <rightJoint>right_wheel_joint</rightJoint>
+                <wheelSeparation>0.3208</wheelSeparation>
+                <wheelDiameter>0.085</wheelDiameter>
+                <wheelAcceleration>1.0</wheelAcceleration>
+                <wheelTorque>20</wheelTorque>
+                <commandTopic>cmd_vel</commandTopic>
+                <odometryTopic>odom</odometryTopic>
+                <odometryFrame>odom</odometryFrame>
+                <robotBaseFrame>base_footprint</robotBaseFrame>
+                <odometrySource>1</odometrySource>
+                <publishWheelTF>true</publishWheelTF>
+                <publishOdom>true</publishOdom>
+                <publishWheelJointState>true</publishWheelJointState>
+                <legacyMode>false</legacyMode>
+            </plugin>
+          </gazebo>
     </xacro:macro>
 </robot>

File: descriptions/urdf/volta0/volta.xacro (robot description, xacro)
@@ -23,6 +23,6 @@
 SOFTWARE, EVEN IF ADVISED OF THE POSSIBILITY OF SUCH DAMAGE.
 -->
-<robot name="volta_robot" xmlns:xacro="https://ros.org/wiki/xacro">
-  <xacro:include filename="$(find volta_description)/urdf/volta.urdf.xacro" />
-  <xacro:volta_robot/>
+<robot name="volta_robot_0" xmlns:xacro="https://ros.org/wiki/xacro">
+  <xacro:include filename="$(find descriptions)/urdf/volta0/volta.urdf.xacro" />
+  <xacro:volta_robot_0/>
 </robot>

File: descriptions/urdf/volta0/volta_properties.xacro (robot description, xacro)
@@ -24,5 +24,5 @@
 SOFTWARE, EVEN IF ADVISED OF THE POSSIBILITY OF SUCH DAMAGE.
 -->
-<robot name="volta_robot" xmlns:xacro="https://ros.org/wiki/xacro">
+<robot name="volta_robot_0" xmlns:xacro="https://ros.org/wiki/xacro">
     <material name="blue">
         <color rgba="0 0 0.8 1"/>

File: descriptions/urdf/volta1/components/caster_volta.urdf.xacro (robot description, xacro)
@@ -24,5 +24,5 @@
 SOFTWARE, EVEN IF ADVISED OF THE POSSIBILITY OF SUCH DAMAGE.
 -->
-<robot name="volta_robot" xmlns:xacro="https://ros.org/wiki/xacro">
+<robot name="volta_robot_1" xmlns:xacro="https://ros.org/wiki/xacro">
     <!-- Caster Macro -->
     <xacro:macro name="volta_caster" params="caster_prefix *caster_joint_origin">
@@ -34,5 +34,5 @@
                     <sphere radius="${caster_radius}"/>
                 </geometry>
-                <material name="Black"/>
+                <material name="black"/>
             </visual>
             <collision>

File: descriptions/urdf/volta1/components/wheel_volta.urdf.xacro (robot description, xacro)
@@ -24,5 +24,5 @@
 SOFTWARE, EVEN IF ADVISED OF THE POSSIBILITY OF SUCH DAMAGE.
 -->
-<robot name="volta_robot" xmlns:xacro="https://ros.org/wiki/xacro">
+<robot name="volta_robot_1" xmlns:xacro="https://ros.org/wiki/xacro">
     <!-- Wheel Macro -->
     <xacro:macro name="volta_wheel" params="wheel_prefix *joint_origin">
