Commit message: Simple leader follower working

File: descriptions/urdf/volta1/volta.urdf.xacro (robot description, xacro)
@@ -24,9 +24,9 @@
 SOFTWARE, EVEN IF ADVISED OF THE POSSIBILITY OF SUCH DAMAGE.
 -->
-<robot name="volta_robot" xmlns:xacro="https://ros.org/wiki/xacro">
+<robot name="volta_robot_1" xmlns:xacro="https://ros.org/wiki/xacro">
     <!-- xacro includes -->
-    <xacro:include filename="$(find volta_description)/urdf/volta_properties.xacro"/>
-    <xacro:include filename="$(find volta_description)/urdf/components/wheel_volta.urdf.xacro"/>
-    <xacro:include filename="$(find volta_description)/urdf/components/caster_volta.urdf.xacro"/>
+    <xacro:include filename="$(find descriptions)/urdf/volta1/volta_properties.xacro"/>
+    <xacro:include filename="$(find descriptions)/urdf/volta1/components/wheel_volta.urdf.xacro"/>
+    <xacro:include filename="$(find descriptions)/urdf/volta1/components/caster_volta.urdf.xacro"/>
     <!-- xacro properties -->
     <xacro:property name="PI" value="3.14159"/>
@@ -34,12 +34,12 @@
     <xacro:arg name="robot_namespace" default="/" />
     <xacro:arg name="tf_pre" default=""/>
-    <xacro:arg name="lidar_enabled" default="true"/>
-    <xacro:arg name="rplidar_a3_enabled" default="true"/>
+    <xacro:arg name="lidar_enabled" default="false"/>
+    <xacro:arg name="rplidar_a3_enabled" default="false"/>
     <xacro:arg name="hokuyo_ust_10lx_enabled" default="false"/>
-    <xacro:arg name="imu_enabled" default="true"/>
-    <xacro:arg name="camera_enabled" default="true"/>
-    <xacro:arg name="intel_d435i_enabled" default="true"/>
+    <xacro:arg name="imu_enabled" default="false"/>
+    <xacro:arg name="camera_enabled" default="false"/>
+    <xacro:arg name="intel_d435i_enabled" default="false"/>
     <xacro:arg name="orbbec_astra_pro_enabled" default="false"/>
-    <xacro:macro name="volta_robot">
+    <xacro:macro name="volta_robot_1">
         <!-- Footprint -->
         <link name="footprint"/>
@@ -55,5 +55,5 @@
                 <origin xyz="0 0 0" rpy="0 0 0" />
                 <geometry>
-                    <mesh filename="package://volta_description/meshes/volta.dae"/>
+                    <mesh filename="package://descriptions/meshes/volta.dae"/>
                 </geometry>
             </visual>
@@ -61,5 +61,5 @@
                 <origin xyz="0 0 0" rpy="0 0 0" />
                 <geometry>
-                    <mesh filename="package://volta_description/meshes/volta_logo.dae"/>
+                    <mesh filename="package://descriptions/meshes/volta_logo.dae"/>
                 </geometry>
             </visual>
@@ -67,5 +67,5 @@
                 <origin xyz="0 0 0" rpy="0 0 0" />
                 <geometry>
-                    <mesh filename="package://volta_description/meshes/volta.dae"/>
+                    <mesh filename="package://descriptions/meshes/volta.dae"/>
                 </geometry>
             </collision>
@@ -98,24 +98,44 @@
         <!-- IMU -->
         <xacro:if value="$(arg imu_enabled)">
-            <xacro:include filename="$(find volta_description)/urdf/accessories/imu_volta.urdf.xacro"/>
+            <xacro:include filename="$(find descriptions)/urdf/volta1/accessories/imu_volta.urdf.xacro"/>
             <xacro:imu robot_namespace="$(arg robot_namespace)" tf_pre="$(arg tf_pre)"></xacro:imu>
         </xacro:if>
         <!-- LIDAR -->
         <xacro:if value="$(arg lidar_enabled)">
-            <xacro:include filename="$(find volta_description)/urdf/accessories/lidar_volta.urdf.xacro"/>
+            <xacro:include filename="$(find descriptions)/urdf/volta1/accessories/lidar_volta.urdf.xacro"/>
             <xacro:lidar rplidar_a3_enabled="$(arg rplidar_a3_enabled)" hokuyo_ust_10lx_enabled="$(arg hokuyo_ust_10lx_enabled)" robot_namespace="$(arg robot_namespace)">  </xacro:lidar>
         </xacro:if>
         <!-- Camera -->
         <xacro:if value="$(arg camera_enabled)">
-            <xacro:include filename="$(find volta_description)/urdf/accessories/camera_volta.urdf.xacro"/>
+            <xacro:include filename="$(find descriptions)/urdf/volta1/accessories/camera_volta.urdf.xacro"/>
             <xacro:camera_ intel_d435i_enabled="$(arg intel_d435i_enabled)" orbbec_astra_pro_enabled="$(arg orbbec_astra_pro_enabled)" robot_namespace="$(arg robot_namespace)"></xacro:camera_>
         </xacro:if>
         <!-- Robot Gazebo tag -->
-        <gazebo>
+        <!-- <gazebo>
             <plugin name="gazebo_ros_control" filename="libgazebo_ros_control.so">
                 <robotNamespace>$(arg robot_namespace)</robotNamespace>
                 <robotSimType>gazebo_ros_control/DefaultRobotHWSim</robotSimType>
             </plugin>
-        </gazebo>
+        </gazebo> -->
+        <gazebo>
+            <plugin name="differential_drive_controller" filename="libgazebo_ros_diff_drive.so">
+                <updateRate>20</updateRate>
+                <leftJoint>left_wheel_joint</leftJoint>
+                <rightJoint>right_wheel_joint</rightJoint>
+                <wheelSeparation>0.3208</wheelSeparation>
+                <wheelDiameter>0.085</wheelDiameter>
+                <wheelAcceleration>1.0</wheelAcceleration>
+                <wheelTorque>20</wheelTorque>
+                <commandTopic>cmd_vel</commandTopic>
+                <odometryTopic>odom</odometryTopic>
+                <odometryFrame>odom</odometryFrame>
+                <robotBaseFrame>base_footprint</robotBaseFrame>
+                <odometrySource>1</odometrySource>
+                <publishWheelTF>true</publishWheelTF>
+                <publishOdom>true</publishOdom>
+                <publishWheelJointState>true</publishWheelJointState>
+                <legacyMode>false</legacyMode>
+            </plugin>
+          </gazebo>
     </xacro:macro>
 </robot>

File: descriptions/urdf/volta1/volta.xacro (robot description, xacro)
@@ -23,6 +23,6 @@
 SOFTWARE, EVEN IF ADVISED OF THE POSSIBILITY OF SUCH DAMAGE.
 -->
-<robot name="volta_robot" xmlns:xacro="https://ros.org/wiki/xacro">
-  <xacro:include filename="$(find volta_description)/urdf/volta.urdf.xacro" />
-  <xacro:volta_robot/>
+<robot name="volta_robot_1" xmlns:xacro="https://ros.org/wiki/xacro">
+  <xacro:include filename="$(find descriptions)/urdf/volta1/volta.urdf.xacro" />
+  <xacro:volta_robot_1/>
 </robot>

File: descriptions/urdf/volta1/volta_properties.xacro (robot description, xacro)
@@ -24,5 +24,5 @@
 SOFTWARE, EVEN IF ADVISED OF THE POSSIBILITY OF SUCH DAMAGE.
 -->
-<robot name="volta_robot" xmlns:xacro="https://ros.org/wiki/xacro">
+<robot name="volta_robot_1" xmlns:xacro="https://ros.org/wiki/xacro">
     <material name="blue">
         <color rgba="0 0 0.8 1"/>

Commit message: Modular Code: Single follower Create single python script for follower robot (Use arguments)

File: descriptions/urdf/volta/accessories/camera_volta.urdf.xacro (robot description, xacro)
@@ -24,5 +24,5 @@
 SOFTWARE, EVEN IF ADVISED OF THE POSSIBILITY OF SUCH DAMAGE.
 -->
-<robot name="volta" xmlns:xacro="https://ros.org/wiki/xacro">
+<robot name="volta_robot" xmlns:xacro="https://ros.org/wiki/xacro">
     <xacro:macro name="camera_" params="frame:=camera topic:=camera info_topic:=camera_info update_rate:=50 intel_d435i_enabled:=true orbbec_astra_pro_enabled:=false robot_namespace:=/">
         <xacro:if value="${intel_d435i_enabled}">

File: descriptions/urdf/volta/accessories/imu_volta.urdf.xacro (robot description, xacro)
@@ -24,5 +24,5 @@
 SOFTWARE, EVEN IF ADVISED OF THE POSSIBILITY OF SUCH DAMAGE.
 -->
-<robot name="volta" xmlns:xacro="https://ros.org/wiki/xacro">
+<robot name="volta_robot" xmlns:xacro="https://ros.org/wiki/xacro">
     <xacro:macro name="imu" params="frame:=imu topic:=imu/data update_rate:=50 robot_namespace:=/ tf_pre:=/">
         <joint name="${frame}_joint" type="fixed">

File: descriptions/urdf/volta/accessories/lidar_volta.urdf.xacro (robot description, xacro)
@@ -24,7 +24,7 @@
 SOFTWARE, EVEN IF ADVISED OF THE POSSIBILITY OF SUCH DAMAGE.
 -->
-<robot name="volta" xmlns:xacro="https://ros.org/wiki/xacro">
+<robot name="volta_robot" xmlns:xacro="https://ros.org/wiki/xacro">
   <xacro:macro name="lidar" params="frame:=lidar topic:=scan_filtered sample_size:=271 update_rate:=50
-                 min_angle:=-1.57 max_angle:=1.57 min_range:=0.5 max_range:=10.0 rplidar_a3_enabled:=true hokuyo_ust_10lx_enabled:=false robot_namespace:=/">
+                 min_angle:=-3.14159 max_angle:=3.14159 min_range:=0.5 max_range:=10.0 rplidar_a3_enabled:=true hokuyo_ust_10lx_enabled:=false robot_namespace:=/">
       <xacro:if value="${rplidar_a3_enabled}">
         <!-- RPLidar mount x position -->
@@ -93,5 +93,5 @@
           <always_on>true</always_on>
           <pose>0 0 0 0 0 0</pose>
-          <visualize>false</visualize>
+          <visualize>true</visualize>
           <update_rate>${update_rate}</update_rate>
           <ray>

File: descriptions/urdf/volta/components/caster_volta.urdf.xacro (robot description, xacro)
@@ -24,5 +24,5 @@
 SOFTWARE, EVEN IF ADVISED OF THE POSSIBILITY OF SUCH DAMAGE.
 -->
-<robot name="volta_robot" xmlns:xacro="https://ros.org/wiki/xacro">
+<robot name="volta_robot_0" xmlns:xacro="https://ros.org/wiki/xacro">
     <!-- Caster Macro -->
     <xacro:macro name="volta_caster" params="caster_prefix *caster_joint_origin">

File: descriptions/urdf/volta/volta.urdf.xacro (robot description, xacro)
@@ -34,6 +34,6 @@
     <xacro:arg name="robot_namespace" default="/" />
     <xacro:arg name="tf_pre" default=""/>
-    <xacro:arg name="lidar_enabled" default="false"/>
-    <xacro:arg name="rplidar_a3_enabled" default="false"/>
+    <xacro:arg name="lidar_enabled" default="true"/>
+    <xacro:arg name="rplidar_a3_enabled" default="true"/>
     <xacro:arg name="hokuyo_ust_10lx_enabled" default="false"/>
     <xacro:arg name="imu_enabled" default="false"/>
@@ -41,5 +41,5 @@
     <xacro:arg name="intel_d435i_enabled" default="false"/>
     <xacro:arg name="orbbec_astra_pro_enabled" default="false"/>
-    <xacro:macro name="volta_robot">
+    <xacro:macro name="volta_robot" params="robot_namespace:=/">
         <!-- Footprint -->
         <link name="footprint"/>
@@ -112,10 +112,30 @@
         </xacro:if>
         <!-- Robot Gazebo tag -->
-        <gazebo>
+        <!-- <gazebo>
             <plugin name="gazebo_ros_control" filename="libgazebo_ros_control.so">
                 <robotNamespace>$(arg robot_namespace)</robotNamespace>
                 <robotSimType>gazebo_ros_control/DefaultRobotHWSim</robotSimType>
             </plugin>
-        </gazebo>
+        </gazebo> -->
+        <gazebo>
+            <plugin name="differential_drive_controller" filename="libgazebo_ros_diff_drive.so">
+                <updateRate>20</updateRate>
+                <leftJoint>left_wheel_joint</leftJoint>
+                <rightJoint>right_wheel_joint</rightJoint>
+                <wheelSeparation>0.3208</wheelSeparation>
+                <wheelDiameter>0.085</wheelDiameter>
+                <wheelAcceleration>1.0</wheelAcceleration>
+                <wheelTorque>20</wheelTorque>
+                <commandTopic>cmd_vel</commandTopic>
+                <odometryTopic>odom</odometryTopic>
+                <odometryFrame>odom</odometryFrame>
+                <robotBaseFrame>base_link</robotBaseFrame>
+                <odometrySource>1</odometrySource>
+                <publishWheelTF>true</publishWheelTF>
+                <publishOdom>true</publishOdom>
+                <publishWheelJointState>true</publishWheelJointState>
+                <legacyMode>false</legacyMode>
+            </plugin>
+          </gazebo>
     </xacro:macro>
 </robot>

File: descriptions/urdf/volta/volta_0.xacro (robot description, xacro)
@@ -24,5 +24,6 @@
 -->
 <robot name="volta_robot" xmlns:xacro="https://ros.org/wiki/xacro">
+  <xacro:arg name="robot_namespace" default="volta_0" />
   <xacro:include filename="$(find descriptions)/urdf/volta/volta.urdf.xacro" />
-  <xacro:volta_robot/>
+  <xacro:volta_robot robot_namespace="$(arg robot_namespace)"/>
 </robot>

File: descriptions/urdf/volta/volta_1.xacro (robot description, xacro)
@@ -1,3 +1,2 @@
-<?xml version="1.0"?>
 <!--
 Copyright (c) 2020, Botsync Pte. Ltd.
@@ -24,33 +23,7 @@
 SOFTWARE, EVEN IF ADVISED OF THE POSSIBILITY OF SUCH DAMAGE.
 -->
-<robot name="volta_robot_3" xmlns:xacro="https://ros.org/wiki/xacro">
-    <xacro:macro name="imu" params="frame:=imu topic:=imu/data update_rate:=50 robot_namespace:=/ tf_pre:=/">
-        <joint name="${frame}_joint" type="fixed">
-            <parent link="base_link" />
-            <child link="${frame}" />
-            <origin xyz="0 0 ${base_h/2}" rpy="0 0 0" />
-        </joint>
-        <link name="${frame}">
-            <inertial>
-                <mass value="0.001"/>
-                <origin xyz="0 0 0" rpy="0 0 0"/>
-                <inertia ixx="1e-09" ixy="0.0" ixz="0.0" iyy="1e-09" iyz="0.0" izz="1e-09"/>
-            </inertial>
-        </link>
-        <gazebo>
-            <plugin name="imu_plugin" filename="libgazebo_ros_imu.so">
-                <alwaysOn>true</alwaysOn>
-                <robotNamespace>${robot_namespace}</robotNamespace>
-                <updateRate>${update_rate}</updateRate>
-                <bodyName>${frame}</bodyName>
-                <frameId>${tf_pre}${frame}</frameId>
-                <frameName>${tf_pre}${frame}</frameName>
-                <topicName>${topic}</topicName>
-                <xyzOffset>0.0 0.0 0.0</xyzOffset>
-                <rpyOffset>0.0 0.0 0.0</rpyOffset>
-                <headingDrift>0.0005</headingDrift>
-                <gaussianNoise>0.0005</gaussianNoise>
-            </plugin>
-        </gazebo>
-    </xacro:macro>
+<robot name="volta_robot" xmlns:xacro="https://ros.org/wiki/xacro">
+  <xacro:arg name="robot_namespace" default="volta_1" />
+  <xacro:include filename="$(find descriptions)/urdf/volta/volta.urdf.xacro" />
+  <xacro:volta_robot robot_namespace="$(arg robot_namespace)"/>
 </robot>

File: descriptions/urdf/volta/volta_2.xacro (robot description, xacro)
@@ -1,3 +1,2 @@
-<?xml version="1.0"?>
 <!--
 Copyright (c) 2020, Botsync Pte. Ltd.
@@ -24,33 +23,7 @@
 SOFTWARE, EVEN IF ADVISED OF THE POSSIBILITY OF SUCH DAMAGE.
 -->
-<robot name="volta" xmlns:xacro="https://ros.org/wiki/xacro">
-    <xacro:macro name="imu" params="frame:=imu topic:=imu/data update_rate:=50 robot_namespace:=/ tf_pre:=/">
-        <joint name="${frame}_joint" type="fixed">
-            <parent link="base_link" />
-            <child link="${frame}" />
-            <origin xyz="0 0 ${base_h/2}" rpy="0 0 0" />
-        </joint>
-        <link name="${frame}">
-            <inertial>
-                <mass value="0.001"/>
-                <origin xyz="0 0 0" rpy="0 0 0"/>
-                <inertia ixx="1e-09" ixy="0.0" ixz="0.0" iyy="1e-09" iyz="0.0" izz="1e-09"/>
-            </inertial>
-        </link>
-        <gazebo>
-            <plugin name="imu_plugin" filename="libgazebo_ros_imu.so">
-                <alwaysOn>true</alwaysOn>
-                <robotNamespace>${robot_namespace}</robotNamespace>
-                <updateRate>${update_rate}</updateRate>
-                <bodyName>${frame}</bodyName>
-                <frameId>${tf_pre}${frame}</frameId>
-                <frameName>${tf_pre}${frame}</frameName>
-                <topicName>${topic}</topicName>
-                <xyzOffset>0.0 0.0 0.0</xyzOffset>
-                <rpyOffset>0.0 0.0 0.0</rpyOffset>
-                <headingDrift>0.0005</headingDrift>
-                <gaussianNoise>0.0005</gaussianNoise>
-            </plugin>
-        </gazebo>
-    </xacro:macro>
+<robot name="volta_robot" xmlns:xacro="https://ros.org/wiki/xacro">
+  <xacro:arg name="robot_namespace" default="volta_2" />
+  <xacro:include filename="$(find descriptions)/urdf/volta/volta.urdf.xacro" />
+  <xacro:volta_robot robot_namespace="$(arg robot_namespace)"/>
 </robot>

File: descriptions/urdf/volta/volta_3.xacro (robot description, xacro)
@@ -23,6 +23,7 @@
 SOFTWARE, EVEN IF ADVISED OF THE POSSIBILITY OF SUCH DAMAGE.
 -->
-<robot name="volta_robot_0" xmlns:xacro="https://ros.org/wiki/xacro">
-  <xacro:include filename="$(find descriptions)/urdf/volta0/volta.urdf.xacro" />
-  <xacro:volta_robot_0/>
+<robot name="volta_robot" xmlns:xacro="https://ros.org/wiki/xacro">
+  <xacro:arg name="robot_namespace" default="volta_3" />
+  <xacro:include filename="$(find descriptions)/urdf/volta/volta.urdf.xacro" />
+  <xacro:volta_robot robot_namespace="$(arg robot_namespace)"/>
 </robot>
