Commit message: Modular Code structure Done

File: descriptions/urdf/volta/accessories/lidar_volta.urdf.xacro (robot description, xacro)
@@ -52,5 +52,5 @@
         <!-- lidar joint -->
         <joint name="lidar_joint" type="fixed">
-            <origin xyz="${lidar_joint_x} ${lidar_joint_y} ${lidar_joint_z + 0.03}" rpy="0 0 0" />
+            <origin xyz="${lidar_joint_x} ${lidar_joint_y} ${lidar_joint_z + 0.03 + 0.2}" rpy="0 0 0" />
             <parent link="base_link" />
             <child link="${frame}" />

Commit message: Distinct aruco marker added on each robot

File: descriptions/urdf/volta/accessories/lidar_volta.urdf.xacro (robot description, xacro)
@@ -52,5 +52,5 @@
         <!-- lidar joint -->
         <joint name="lidar_joint" type="fixed">
-            <origin xyz="${lidar_joint_x} ${lidar_joint_y} ${lidar_joint_z + 0.03 + 0.2}" rpy="0 0 0" />
+            <origin xyz="${lidar_joint_x} ${lidar_joint_y} ${lidar_joint_z + 0.03 + 0.15}" rpy="0 0 0" />
             <parent link="base_link" />
             <child link="${frame}" />
@@ -93,5 +93,5 @@
           <always_on>true</always_on>
           <pose>0 0 0 0 0 0</pose>
-          <visualize>true</visualize>
+          <visualize>false</visualize>
           <update_rate>${update_rate}</update_rate>
           <ray>

File: descriptions/urdf/volta/volta.urdf.xacro (robot description, xacro)
@@ -38,6 +38,6 @@
     <xacro:arg name="hokuyo_ust_10lx_enabled" default="false"/>
     <xacro:arg name="imu_enabled" default="false"/>
-    <xacro:arg name="camera_enabled" default="false"/>
-    <xacro:arg name="intel_d435i_enabled" default="false"/>
+    <xacro:arg name="camera_enabled" default="true"/>
+    <xacro:arg name="intel_d435i_enabled" default="true"/>
     <xacro:arg name="orbbec_astra_pro_enabled" default="false"/>
     <xacro:macro name="volta_robot" params="robot_namespace:=/">
@@ -106,4 +106,6 @@
             <xacro:lidar rplidar_a3_enabled="$(arg rplidar_a3_enabled)" hokuyo_ust_10lx_enabled="$(arg hokuyo_ust_10lx_enabled)" robot_namespace="$(arg robot_namespace)">  </xacro:lidar>
         </xacro:if>
+        <xacro:include filename="$(find descriptions)/urdf/volta/accessories/aruco_marker.urdf.xacro"/>
+        <xacro:aruco_marker robot_namespace="$(arg robot_namespace)">  </xacro:aruco_marker>
         <!-- Camera -->
         <xacro:if value="$(arg camera_enabled)">

Commit message: Updated lidar properties

File: descriptions/urdf/volta/accessories/lidar_volta.urdf.xacro (robot description, xacro)
@@ -25,6 +25,7 @@
 -->
 <robot name="volta_robot" xmlns:xacro="https://ros.org/wiki/xacro">
-  <xacro:macro name="lidar" params="frame:=lidar topic:=scan_filtered sample_size:=271 update_rate:=50
-                 min_angle:=-3.14159 max_angle:=3.14159 min_range:=0.5 max_range:=10.0 rplidar_a3_enabled:=true hokuyo_ust_10lx_enabled:=false robot_namespace:=/">
+  <xacro:macro name="lidar" params="frame:=lidar topic:=scan_filtered sample_size:=271 update_rate:=120
+                 min_angle:=-1.75 max_angle:=1.75 min_range:=0.1 max_range:=10.0 rplidar_a3_enabled:=true hokuyo_ust_10lx_enabled:=false robot_namespace:=/">
+                 <!-- min_angle:=-3.14159 max_angle:=3.14159 min_range:=0.5 max_range:=10.0 rplidar_a3_enabled:=true hokuyo_ust_10lx_enabled:=false robot_namespace:=/"> -->
       <xacro:if value="${rplidar_a3_enabled}">
         <!-- RPLidar mount x position -->

Commit message: Ready for demos

File: descriptions/urdf/volta/accessories/lidar_volta.urdf.xacro (robot description, xacro)
@@ -26,5 +26,6 @@
 <robot name="volta_robot" xmlns:xacro="https://ros.org/wiki/xacro">
   <xacro:macro name="lidar" params="frame:=lidar topic:=scan_filtered sample_size:=271 update_rate:=120
-                 min_angle:=-3.14159 max_angle:=3.14159 min_range:=0.5 max_range:=10.0 rplidar_a3_enabled:=true hokuyo_ust_10lx_enabled:=false robot_namespace:=/">
+                 min_angle:=-3.14159 max_angle:=3.14159 min_range:=0.05 max_range:=10.0 rplidar_a3_enabled:=true hokuyo_ust_10lx_enabled:=false robot_namespace:=/">
+                 <!-- min_angle:=-3.14159 max_angle:=3.14159 min_range:=0.5 max_range:=10.0 rplidar_a3_enabled:=true hokuyo_ust_10lx_enabled:=false robot_namespace:=/"> -->
                  <!-- min_angle:=-1.75 max_angle:=1.75 min_range:=0.1 max_range:=10.0 rplidar_a3_enabled:=true hokuyo_ust_10lx_enabled:=false robot_namespace:=/"> -->
       <xacro:if value="${rplidar_a3_enabled}">
@@ -53,6 +54,6 @@
         <!-- lidar joint -->
         <joint name="lidar_joint" type="fixed">
-            <origin xyz="${lidar_joint_x} ${lidar_joint_y} ${lidar_joint_z + 0.03}" rpy="0 0 0" />
-            <!-- <origin xyz="${lidar_joint_x} ${lidar_joint_y} ${lidar_joint_z + 0.03 + 0.15}" rpy="0 0 0" /> -->
+            <!-- <origin xyz="${lidar_joint_x} ${lidar_joint_y} ${lidar_joint_z + 0.03}" rpy="0 0 0" /> -->
+            <origin xyz="${lidar_joint_x} ${lidar_joint_y} ${lidar_joint_z + 0.03 + 0.15}" rpy="0 0 0" />
             <parent link="base_link" />
             <child link="${frame}" />
@@ -95,5 +96,5 @@
           <always_on>true</always_on>
           <pose>0 0 0 0 0 0</pose>
-          <visualize>true</visualize>
+          <visualize>false</visualize>
           <update_rate>${update_rate}</update_rate>
           <ray>
