Commit message: Robot ID detection using Aruco Marker

File: descriptions/urdf/volta/accessories/aruco_marker.urdf.xacro (robot description, xacro)
@@ -85,5 +85,5 @@
 		</link>
 		<joint name="aruco_marker_joint_back" type="fixed">
-			<origin xyz="-0.27 0 0.08" rpy="0 ${PI/2} 0" />
+			<origin xyz="-0.27 0 0.08" rpy="0 -${PI/2} 0" />
 			<parent link="base_link" />
 			<child link="${frame}_back" />
@@ -100,5 +100,5 @@
 		</joint>
 		<joint name="aruco_marker_joint_left" type="fixed">
-			<origin xyz="0 0.2 0.08" rpy="${PI/2} 0 0" />
+			<origin xyz="0 0.2 0.08" rpy="-${PI/2} 0 0" />
 			<parent link="base_link" />
 			<child link="${frame}_left" />

Commit message: Testing convoy with 7 robots

File: descriptions/urdf/volta/accessories/aruco_marker.urdf.xacro (robot description, xacro)
@@ -27,5 +27,4 @@
 	<xacro:property name="PI" value="3.14159" />
 	<xacro:macro name="aruco_marker" params="frame:=aruco_marker robot_namespace:=/">
-		<xacro:property name="lidar_joint_x" value="0.1995" />
 		<link name="${frame}_back">
 			<visual>
@@ -85,20 +84,20 @@
 		</link>
 		<joint name="aruco_marker_joint_back" type="fixed">
-			<origin xyz="-0.27 0 0.08" rpy="0 -${PI/2} 0" />
+			<origin xyz="-0.27 0 0.35" rpy="0 -${PI/2} 0" />
 			<parent link="base_link" />
 			<child link="${frame}_back" />
 		</joint>
 		<joint name="aruco_marker_joint_front" type="fixed">
-			<origin xyz="0.27 0 0.08" rpy="0 ${PI/2} 0" />
+			<origin xyz="0.27 0 0.35" rpy="0 ${PI/2} 0" />
 			<parent link="base_link" />
 			<child link="${frame}_front" />
 		</joint>
 		<joint name="aruco_marker_joint_right" type="fixed">
-			<origin xyz="0 -0.2 0.08" rpy="${PI/2} 0 0" />
+			<origin xyz="0 -0.2 0.35" rpy="${PI/2} 0 0" />
 			<parent link="base_link" />
 			<child link="${frame}_right" />
 		</joint>
 		<joint name="aruco_marker_joint_left" type="fixed">
-			<origin xyz="0 0.2 0.08" rpy="-${PI/2} 0 0" />
+			<origin xyz="0 0.2 0.35" rpy="-${PI/2} 0 0" />
 			<parent link="base_link" />
 			<child link="${frame}_left" />

File: descriptions/urdf/volta/accessories/lidar_volta.urdf.xacro (robot description, xacro)
@@ -52,5 +52,6 @@
         <!-- lidar joint -->
         <joint name="lidar_joint" type="fixed">
-            <origin xyz="${lidar_joint_x} ${lidar_joint_y} ${lidar_joint_z + 0.03 + 0.15}" rpy="0 0 0" />
+            <origin xyz="${lidar_joint_x} ${lidar_joint_y} ${lidar_joint_z + 0.03}" rpy="0 0 0" />
+            <!-- <origin xyz="${lidar_joint_x} ${lidar_joint_y} ${lidar_joint_z + 0.03 + 0.15}" rpy="0 0 0" /> -->
             <parent link="base_link" />
             <child link="${frame}" />

Commit message: Updated conditions for navigation

File: descriptions/urdf/volta/accessories/aruco_marker.urdf.xacro (robot description, xacro)
@@ -27,79 +27,231 @@
 	<xacro:property name="PI" value="3.14159" />
 	<xacro:macro name="aruco_marker" params="frame:=aruco_marker robot_namespace:=/">
-		<link name="${frame}_back">
-			<visual>
-				<origin xyz="0 0 0" />
-				<geometry>
-					<mesh filename="package://descriptions/urdf/volta/meshes/${robot_namespace}_aruco.dae" scale="0.5 0.5 0.5"/>
-				</geometry>
-			</visual>
-			<collision>
-				<origin xyz="0 0 0" />
-				<geometry>
-					<mesh filename="package://descriptions/urdf/volta/meshes/${robot_namespace}_aruco.dae" scale="0.5 0.5 0.5"/>
-				</geometry>
-			</collision>
-		</link>
-		<link name="${frame}_front">
-			<visual>
-				<origin xyz="0 0 0" />
-				<geometry>
-					<mesh filename="package://descriptions/urdf/volta/meshes/${robot_namespace}_aruco.dae" scale="0.5 0.5 0.5"/>
-				</geometry>
-			</visual>
-			<collision>
-				<origin xyz="0 0 0" />
-				<geometry>
-					<mesh filename="package://descriptions/urdf/volta/meshes/${robot_namespace}_aruco.dae" scale="0.5 0.5 0.5"/>
-				</geometry>
-			</collision>
-		</link>
-		<link name="${frame}_right">
-			<visual>
-				<origin xyz="0 0 0" />
-				<geometry>
-					<mesh filename="package://descriptions/urdf/volta/meshes/${robot_namespace}_aruco.dae" scale="0.5 0.5 0.5"/>
-				</geometry>
-			</visual>
-			<collision>
-				<origin xyz="0 0 0" />
-				<geometry>
-					<mesh filename="package://descriptions/urdf/volta/meshes/${robot_namespace}_aruco.dae" scale="0.5 0.5 0.5"/>
-				</geometry>
-			</collision>
-		</link>
-		<link name="${frame}_left">
-			<visual>
-				<origin xyz="0 0 0" />
-				<geometry>
-					<mesh filename="package://descriptions/urdf/volta/meshes/${robot_namespace}_aruco.dae" scale="0.5 0.5 0.5"/>
-				</geometry>
-			</visual>
-			<collision>
-				<origin xyz="0 0 0" />
-				<geometry>
-					<mesh filename="package://descriptions/urdf/volta/meshes/${robot_namespace}_aruco.dae" scale="0.5 0.5 0.5"/>
-				</geometry>
-			</collision>
-		</link>
-		<joint name="aruco_marker_joint_back" type="fixed">
-			<origin xyz="-0.27 0 0.35" rpy="0 -${PI/2} 0" />
-			<parent link="base_link" />
-			<child link="${frame}_back" />
-		</joint>
-		<joint name="aruco_marker_joint_front" type="fixed">
-			<origin xyz="0.27 0 0.35" rpy="0 ${PI/2} 0" />
-			<parent link="base_link" />
-			<child link="${frame}_front" />
-		</joint>
-		<joint name="aruco_marker_joint_right" type="fixed">
-			<origin xyz="0 -0.2 0.35" rpy="${PI/2} 0 0" />
-			<parent link="base_link" />
-			<child link="${frame}_right" />
-		</joint>
-		<joint name="aruco_marker_joint_left" type="fixed">
-			<origin xyz="0 0.2 0.35" rpy="-${PI/2} 0 0" />
-			<parent link="base_link" />
-			<child link="${frame}_left" />
+		<link name="${frame}_back_0">
+			<visual>
+				<origin xyz="0 0 0" />
+				<geometry>
+					<mesh filename="package://descriptions/urdf/volta/meshes/${robot_namespace}_aruco.dae" scale="0.25 0.25 0.25"/>
+				</geometry>
+			</visual>
+			<collision>
+				<origin xyz="0 0 0" />
+				<geometry>
+					<mesh filename="package://descriptions/urdf/volta/meshes/${robot_namespace}_aruco.dae" scale="0.25 0.25 0.25"/>
+				</geometry>
+			</collision>
+		</link>
+		<link name="${frame}_back_1">
+			<visual>
+				<origin xyz="0 0 0" />
+				<geometry>
+					<mesh filename="package://descriptions/urdf/volta/meshes/${robot_namespace}_aruco.dae" scale="0.25 0.25 0.25"/>
+				</geometry>
+			</visual>
+			<collision>
+				<origin xyz="0 0 0" />
+				<geometry>
+					<mesh filename="package://descriptions/urdf/volta/meshes/${robot_namespace}_aruco.dae" scale="0.25 0.25 0.25"/>
+				</geometry>
+			</collision>
+		</link>
+		<link name="${frame}_back_2">
+			<visual>
+				<origin xyz="0 0 0" />
+				<geometry>
+					<mesh filename="package://descriptions/urdf/volta/meshes/${robot_namespace}_aruco.dae" scale="0.25 0.25 0.25"/>
+				</geometry>
+			</visual>
+			<collision>
+				<origin xyz="0 0 0" />
+				<geometry>
+					<mesh filename="package://descriptions/urdf/volta/meshes/${robot_namespace}_aruco.dae" scale="0.25 0.25 0.25"/>
+				</geometry>
+			</collision>
+		</link>
+		<link name="${frame}_front_0">
+			<visual>
+				<origin xyz="0 0 0" />
+				<geometry>
+					<mesh filename="package://descriptions/urdf/volta/meshes/${robot_namespace}_aruco.dae" scale="0.25 0.25 0.25"/>
+				</geometry>
+			</visual>
+			<collision>
+				<origin xyz="0 0 0" />
+				<geometry>
+					<mesh filename="package://descriptions/urdf/volta/meshes/${robot_namespace}_aruco.dae" scale="0.25 0.25 0.25"/>
+				</geometry>
+			</collision>
+		</link>
+		<link name="${frame}_front_1">
+			<visual>
+				<origin xyz="0 0 0" />
+				<geometry>
+					<mesh filename="package://descriptions/urdf/volta/meshes/${robot_namespace}_aruco.dae" scale="0.25 0.25 0.25"/>
+				</geometry>
+			</visual>
+			<collision>
+				<origin xyz="0 0 0" />
+				<geometry>
+					<mesh filename="package://descriptions/urdf/volta/meshes/${robot_namespace}_aruco.dae" scale="0.25 0.25 0.25"/>
+				</geometry>
+			</collision>
+		</link>
+		<link name="${frame}_front_2">
+			<visual>
+				<origin xyz="0 0 0" />
+				<geometry>
+					<mesh filename="package://descriptions/urdf/volta/meshes/${robot_namespace}_aruco.dae" scale="0.25 0.25 0.25"/>
+				</geometry>
+			</visual>
+			<collision>
+				<origin xyz="0 0 0" />
+				<geometry>
+					<mesh filename="package://descriptions/urdf/volta/meshes/${robot_namespace}_aruco.dae" scale="0.25 0.25 0.25"/>
+				</geometry>
+			</collision>
+		</link>
+		<link name="${frame}_right_0">
+			<visual>
+				<origin xyz="0 0 0" />
+				<geometry>
+					<mesh filename="package://descriptions/urdf/volta/meshes/${robot_namespace}_aruco.dae" scale="0.25 0.25 0.25"/>
+				</geometry>
+			</visual>
+			<collision>
+				<origin xyz="0 0 0" />
+				<geometry>
+					<mesh filename="package://descriptions/urdf/volta/meshes/${robot_namespace}_aruco.dae" scale="0.25 0.25 0.25"/>
+				</geometry>
+			</collision>
+		</link>
+		<link name="${frame}_right_1">
+			<visual>
+				<origin xyz="0 0 0" />
+				<geometry>
+					<mesh filename="package://descriptions/urdf/volta/meshes/${robot_namespace}_aruco.dae" scale="0.25 0.25 0.25"/>
+				</geometry>
+			</visual>
+			<collision>
+				<origin xyz="0 0 0" />
+				<geometry>
+					<mesh filename="package://descriptions/urdf/volta/meshes/${robot_namespace}_aruco.dae" scale="0.25 0.25 0.25"/>
+				</geometry>
+			</collision>
+		</link>
+		<link name="${frame}_right_2">
+			<visual>
+				<origin xyz="0 0 0" />
+				<geometry>
+					<mesh filename="package://descriptions/urdf/volta/meshes/${robot_namespace}_aruco.dae" scale="0.25 0.25 0.25"/>
+				</geometry>
+			</visual>
+			<collision>
+				<origin xyz="0 0 0" />
+				<geometry>
+					<mesh filename="package://descriptions/urdf/volta/meshes/${robot_namespace}_aruco.dae" scale="0.25 0.25 0.25"/>
+				</geometry>
+			</collision>
+		</link>
+		<link name="${frame}_left_0">
+			<visual>
+				<origin xyz="0 0 0" />
+				<geometry>
+					<mesh filename="package://descriptions/urdf/volta/meshes/${robot_namespace}_aruco.dae" scale="0.25 0.25 0.25"/>
+				</geometry>
+			</visual>
+			<collision>
+				<origin xyz="0 0 0" />
+				<geometry>
+					<mesh filename="package://descriptions/urdf/volta/meshes/${robot_namespace}_aruco.dae" scale="0.25 0.25 0.25"/>
+				</geometry>
+			</collision>
+		</link>
+		<link name="${frame}_left_1">
+			<visual>
+				<origin xyz="0 0 0" />
+				<geometry>
+					<mesh filename="package://descriptions/urdf/volta/meshes/${robot_namespace}_aruco.dae" scale="0.25 0.25 0.25"/>
+				</geometry>
+			</visual>
+			<collision>
+				<origin xyz="0 0 0" />
+				<geometry>
+					<mesh filename="package://descriptions/urdf/volta/meshes/${robot_namespace}_aruco.dae" scale="0.25 0.25 0.25"/>
+				</geometry>
+			</collision>
+		</link>
+		<link name="${frame}_left_2">
+			<visual>
+				<origin xyz="0 0 0" />
+				<geometry>
+					<mesh filename="package://descriptions/urdf/volta/meshes/${robot_namespace}_aruco.dae" scale="0.25 0.25 0.25"/>
+				</geometry>
+			</visual>
+			<collision>
+				<origin xyz="0 0 0" />
+				<geometry>
+					<mesh filename="package://descriptions/urdf/volta/meshes/${robot_namespace}_aruco.dae" scale="0.25 0.25 0.25"/>
+				</geometry>
+			</collision>
+		</link>
+		<joint name="aruco_marker_joint_back_0" type="fixed">
+			<origin xyz="-0.27 0 0.15" rpy="0 -${PI/2} 0" />
+			<parent link="base_link" />
+			<child link="${frame}_back_0" />
+		</joint>
+		<joint name="aruco_marker_joint_back_1" type="fixed">
+			<origin xyz="-0.27 -0.125 0.15" rpy="0 -${PI/2} 0" />
+			<parent link="base_link" />
+			<child link="${frame}_back_1" />
+		</joint>
+		<joint name="aruco_marker_joint_back_2" type="fixed">
+			<origin xyz="-0.27 0.125 0.15" rpy="0 -${PI/2} 0" />
+			<parent link="base_link" />
+			<child link="${frame}_back_2" />
+		</joint>
+		<joint name="aruco_marker_joint_front_0" type="fixed">
+			<origin xyz="0.27 0 0.15" rpy="0 ${PI/2} 0" />
+			<parent link="base_link" />
+			<child link="${frame}_front_0" />
+		</joint>
+		<joint name="aruco_marker_joint_front_1" type="fixed">
+			<origin xyz="0.27 -0.125 0.15" rpy="0 ${PI/2} 0" />
+			<parent link="base_link" />
+			<child link="${frame}_front_1" />
+		</joint>
+		<joint name="aruco_marker_joint_front_2" type="fixed">
+			<origin xyz="0.27 0.125 0.15" rpy="0 ${PI/2} 0" />
+			<parent link="base_link" />
+			<child link="${frame}_front_2" />
+		</joint>
+		<joint name="aruco_marker_joint_right_0" type="fixed">
+			<origin xyz="0 -0.2 0.15" rpy="${PI/2} 0 0" />
+			<parent link="base_link" />
+			<child link="${frame}_right_0" />
+		</joint>
+		<joint name="aruco_marker_joint_right_1" type="fixed">
+			<origin xyz="-0.2 -0.2 0.15" rpy="${PI/2} 0 0" />
+			<parent link="base_link" />
+			<child link="${frame}_right_1" />
+		</joint>
+		<joint name="aruco_marker_joint_right_2" type="fixed">
+			<origin xyz="0.2 -0.2 0.15" rpy="${PI/2} 0 0" />
+			<parent link="base_link" />
+			<child link="${frame}_right_2" />
+		</joint>
+		<joint name="aruco_marker_joint_left_0" type="fixed">
+			<origin xyz="0 0.2 0.15" rpy="-${PI/2} 0 0" />
+			<parent link="base_link" />
+			<child link="${frame}_left_0" />
+		</joint>
+		<joint name="aruco_marker_joint_left_1" type="fixed">
+			<origin xyz="-0.2 0.2 0.15" rpy="-${PI/2} 0 0" />
+			<parent link="base_link" />
+			<child link="${frame}_left_1" />
+		</joint>
+		<joint name="aruco_marker_joint_left_2" type="fixed">
+			<origin xyz="0.2 0.2 0.15" rpy="-${PI/2} 0 0" />
+			<parent link="base_link" />
+			<child link="${frame}_left_2" />
 		</joint>
 		<gazebo reference="${frame}_back"/>

File: descriptions/urdf/volta/volta.urdf.xacro (robot description, xacro)
@@ -38,6 +38,6 @@
     <xacro:arg name="hokuyo_ust_10lx_enabled" default="false"/>
     <xacro:arg name="imu_enabled" default="false"/>
-    <xacro:arg name="camera_enabled" default="true"/>
-    <xacro:arg name="intel_d435i_enabled" default="true"/>
+    <xacro:arg name="camera_enabled" default="false"/>
+    <xacro:arg name="intel_d435i_enabled" default="false"/>
     <xacro:arg name="orbbec_astra_pro_enabled" default="false"/>
     <xacro:macro name="volta_robot" params="robot_namespace:=/">
@@ -106,6 +106,6 @@
             <xacro:lidar rplidar_a3_enabled="$(arg rplidar_a3_enabled)" hokuyo_ust_10lx_enabled="$(arg hokuyo_ust_10lx_enabled)" robot_namespace="$(arg robot_namespace)">  </xacro:lidar>
         </xacro:if>
-        <!-- <xacro:include filename="$(find descriptions)/urdf/volta/accessories/aruco_marker.urdf.xacro"/>
-        <xacro:aruco_marker robot_namespace="$(arg robot_namespace)">  </xacro:aruco_marker> -->
+        <xacro:include filename="$(find descriptions)/urdf/volta/accessories/aruco_marker.urdf.xacro"/>
+        <xacro:aruco_marker robot_namespace="$(arg robot_namespace)">  </xacro:aruco_marker>
         <!-- Camera -->
         <xacro:if value="$(arg camera_enabled)">
