Commit message: Added Camera node

File: descriptions/urdf/volta/accessories/aruco_marker.urdf.xacro (robot description, xacro)
@@ -31,11 +31,11 @@
 				<origin xyz="0 0 0" />
 				<geometry>
-					<mesh filename="package://descriptions/urdf/volta/meshes/${robot_namespace}_aruco.dae" scale="0.25 0.25 0.25"/>
-				</geometry>
-			</visual>
-			<collision>
-				<origin xyz="0 0 0" />
-				<geometry>
-					<mesh filename="package://descriptions/urdf/volta/meshes/${robot_namespace}_aruco.dae" scale="0.25 0.25 0.25"/>
+					<mesh filename="package://descriptions/urdf/volta/meshes/${robot_namespace}_aruco.dae" scale="0.3 0.3 0.3"/>
+				</geometry>
+			</visual>
+			<collision>
+				<origin xyz="0 0 0" />
+				<geometry>
+					<mesh filename="package://descriptions/urdf/volta/meshes/${robot_namespace}_aruco.dae" scale="0.3 0.3 0.3"/>
 				</geometry>
 			</collision>
@@ -45,11 +45,11 @@
 				<origin xyz="0 0 0" />
 				<geometry>
-					<mesh filename="package://descriptions/urdf/volta/meshes/${robot_namespace}_aruco.dae" scale="0.25 0.25 0.25"/>
-				</geometry>
-			</visual>
-			<collision>
-				<origin xyz="0 0 0" />
-				<geometry>
-					<mesh filename="package://descriptions/urdf/volta/meshes/${robot_namespace}_aruco.dae" scale="0.25 0.25 0.25"/>
+					<mesh filename="package://descriptions/urdf/volta/meshes/${robot_namespace}_aruco.dae" scale="0.3 0.3 0.3"/>
+				</geometry>
+			</visual>
+			<collision>
+				<origin xyz="0 0 0" />
+				<geometry>
+					<mesh filename="package://descriptions/urdf/volta/meshes/${robot_namespace}_aruco.dae" scale="0.3 0.3 0.3"/>
 				</geometry>
 			</collision>
@@ -59,11 +59,11 @@
 				<origin xyz="0 0 0" />
 				<geometry>
-					<mesh filename="package://descriptions/urdf/volta/meshes/${robot_namespace}_aruco.dae" scale="0.25 0.25 0.25"/>
-				</geometry>
-			</visual>
-			<collision>
-				<origin xyz="0 0 0" />
-				<geometry>
-					<mesh filename="package://descriptions/urdf/volta/meshes/${robot_namespace}_aruco.dae" scale="0.25 0.25 0.25"/>
+					<mesh filename="package://descriptions/urdf/volta/meshes/${robot_namespace}_aruco.dae" scale="0.3 0.3 0.3"/>
+				</geometry>
+			</visual>
+			<collision>
+				<origin xyz="0 0 0" />
+				<geometry>
+					<mesh filename="package://descriptions/urdf/volta/meshes/${robot_namespace}_aruco.dae" scale="0.3 0.3 0.3"/>
 				</geometry>
 			</collision>
@@ -73,11 +73,11 @@
 				<origin xyz="0 0 0" />
 				<geometry>
-					<mesh filename="package://descriptions/urdf/volta/meshes/${robot_namespace}_aruco.dae" scale="0.25 0.25 0.25"/>
-				</geometry>
-			</visual>
-			<collision>
-				<origin xyz="0 0 0" />
-				<geometry>
-					<mesh filename="package://descriptions/urdf/volta/meshes/${robot_namespace}_aruco.dae" scale="0.25 0.25 0.25"/>
+					<mesh filename="package://descriptions/urdf/volta/meshes/${robot_namespace}_aruco.dae" scale="0.3 0.3 0.3"/>
+				</geometry>
+			</visual>
+			<collision>
+				<origin xyz="0 0 0" />
+				<geometry>
+					<mesh filename="package://descriptions/urdf/volta/meshes/${robot_namespace}_aruco.dae" scale="0.3 0.3 0.3"/>
 				</geometry>
 			</collision>
@@ -87,11 +87,11 @@
 				<origin xyz="0 0 0" />
 				<geometry>
-					<mesh filename="package://descriptions/urdf/volta/meshes/${robot_namespace}_aruco.dae" scale="0.25 0.25 0.25"/>
-				</geometry>
-			</visual>
-			<collision>
-				<origin xyz="0 0 0" />
-				<geometry>
-					<mesh filename="package://descriptions/urdf/volta/meshes/${robot_namespace}_aruco.dae" scale="0.25 0.25 0.25"/>
+					<mesh filename="package://descriptions/urdf/volta/meshes/${robot_namespace}_aruco.dae" scale="0.3 0.3 0.3"/>
+				</geometry>
+			</visual>
+			<collision>
+				<origin xyz="0 0 0" />
+				<geometry>
+					<mesh filename="package://descriptions/urdf/volta/meshes/${robot_namespace}_aruco.dae" scale="0.3 0.3 0.3"/>
 				</geometry>
 			</collision>
@@ -101,11 +101,11 @@
 				<origin xyz="0 0 0" />
 				<geometry>
-					<mesh filename="package://descriptions/urdf/volta/meshes/${robot_namespace}_aruco.dae" scale="0.25 0.25 0.25"/>
-				</geometry>
-			</visual>
-			<collision>
-				<origin xyz="0 0 0" />
-				<geometry>
-					<mesh filename="package://descriptions/urdf/volta/meshes/${robot_namespace}_aruco.dae" scale="0.25 0.25 0.25"/>
+					<mesh filename="package://descriptions/urdf/volta/meshes/${robot_namespace}_aruco.dae" scale="0.3 0.3 0.3"/>
+				</geometry>
+			</visual>
+			<collision>
+				<origin xyz="0 0 0" />
+				<geometry>
+					<mesh filename="package://descriptions/urdf/volta/meshes/${robot_namespace}_aruco.dae" scale="0.3 0.3 0.3"/>
 				</geometry>
 			</collision>
@@ -115,11 +115,11 @@
 				<origin xyz="0 0 0" />
 				<geometry>
-					<mesh filename="package://descriptions/urdf/volta/meshes/${robot_namespace}_aruco.dae" scale="0.25 0.25 0.25"/>
-				</geometry>
-			</visual>
-			<collision>
-				<origin xyz="0 0 0" />
-				<geometry>
-					<mesh filename="package://descriptions/urdf/volta/meshes/${robot_namespace}_aruco.dae" scale="0.25 0.25 0.25"/>
+					<mesh filename="package://descriptions/urdf/volta/meshes/${robot_namespace}_aruco.dae" scale="0.3 0.3 0.3"/>
+				</geometry>
+			</visual>
+			<collision>
+				<origin xyz="0 0 0" />
+				<geometry>
+					<mesh filename="package://descriptions/urdf/volta/meshes/${robot_namespace}_aruco.dae" scale="0.3 0.3 0.3"/>
 				</geometry>
 			</collision>
@@ -129,11 +129,11 @@
 				<origin xyz="0 0 0" />
 				<geometry>
-					<mesh filename="package://descriptions/urdf/volta/meshes/${robot_namespace}_aruco.dae" scale="0.25 0.25 0.25"/>
-				</geometry>
-			</visual>
-			<collision>
-				<origin xyz="0 0 0" />
-				<geometry>
-					<mesh filename="package://descriptions/urdf/volta/meshes/${robot_namespace}_aruco.dae" scale="0.25 0.25 0.25"/>
+					<mesh filename="package://descriptions/urdf/volta/meshes/${robot_namespace}_aruco.dae" scale="0.3 0.3 0.3"/>
+				</geometry>
+			</visual>
+			<collision>
+				<origin xyz="0 0 0" />
+				<geometry>
+					<mesh filename="package://descriptions/urdf/volta/meshes/${robot_namespace}_aruco.dae" scale="0.3 0.3 0.3"/>
 				</geometry>
 			</collision>
@@ -143,11 +143,11 @@
 				<origin xyz="0 0 0" />
 				<geometry>
-					<mesh filename="package://descriptions/urdf/volta/meshes/${robot_namespace}_aruco.dae" scale="0.25 0.25 0.25"/>
-				</geometry>
-			</visual>
-			<collision>
-				<origin xyz="0 0 0" />
-				<geometry>
-					<mesh filename="package://descriptions/urdf/volta/meshes/${robot_namespace}_aruco.dae" scale="0.25 0.25 0.25"/>
+					<mesh filename="package://descriptions/urdf/volta/meshes/${robot_namespace}_aruco.dae" scale="0.3 0.3 0.3"/>
+				</geometry>
+			</visual>
+			<collision>
+				<origin xyz="0 0 0" />
+				<geometry>
+					<mesh filename="package://descriptions/urdf/volta/meshes/${robot_namespace}_aruco.dae" scale="0.3 0.3 0.3"/>
 				</geometry>
 			</collision>
@@ -157,11 +157,11 @@
 				<origin xyz="0 0 0" />
 				<geometry>
-					<mesh filename="package://descriptions/urdf/volta/meshes/${robot_namespace}_aruco.dae" scale="0.25 0.25 0.25"/>
-				</geometry>
-			</visual>
-			<collision>
-				<origin xyz="0 0 0" />
-				<geometry>
-					<mesh filename="package://descriptions/urdf/volta/meshes/${robot_namespace}_aruco.dae" scale="0.25 0.25 0.25"/>
+					<mesh filename="package://descriptions/urdf/volta/meshes/${robot_namespace}_aruco.dae" scale="0.3 0.3 0.3"/>
+				</geometry>
+			</visual>
+			<collision>
+				<origin xyz="0 0 0" />
+				<geometry>
+					<mesh filename="package://descriptions/urdf/volta/meshes/${robot_namespace}_aruco.dae" scale="0.3 0.3 0.3"/>
 				</geometry>
 			</collision>
@@ -171,11 +171,11 @@
 				<origin xyz="0 0 0" />
 				<geometry>
-					<mesh filename="package://descriptions/urdf/volta/meshes/${robot_namespace}_aruco.dae" scale="0.25 0.25 0.25"/>
-				</geometry>
-			</visual>
-			<collision>
-				<origin xyz="0 0 0" />
-				<geometry>
-					<mesh filename="package://descriptions/urdf/volta/meshes/${robot_namespace}_aruco.dae" scale="0.25 0.25 0.25"/>
+					<mesh filename="package://descriptions/urdf/volta/meshes/${robot_namespace}_aruco.dae" scale="0.3 0.3 0.3"/>
+				</geometry>
+			</visual>
+			<collision>
+				<origin xyz="0 0 0" />
+				<geometry>
+					<mesh filename="package://descriptions/urdf/volta/meshes/${robot_namespace}_aruco.dae" scale="0.3 0.3 0.3"/>
 				</geometry>
 			</collision>
@@ -185,11 +185,11 @@
 				<origin xyz="0 0 0" />
 				<geometry>
-					<mesh filename="package://descriptions/urdf/volta/meshes/${robot_namespace}_aruco.dae" scale="0.25 0.25 0.25"/>
-				</geometry>
-			</visual>
-			<collision>
-				<origin xyz="0 0 0" />
-				<geometry>
-					<mesh filename="package://descriptions/urdf/volta/meshes/${robot_namespace}_aruco.dae" scale="0.25 0.25 0.25"/>
+					<mesh filename="package://descriptions/urdf/volta/meshes/${robot_namespace}_aruco.dae" scale="0.3 0.3 0.3"/>
+				</geometry>
+			</visual>
+			<collision>
+				<origin xyz="0 0 0" />
+				<geometry>
+					<mesh filename="package://descriptions/urdf/volta/meshes/${robot_namespace}_aruco.dae" scale="0.3 0.3 0.3"/>
 				</geometry>
 			</collision>
