Commit message: Ready to test communication based formation

File: descriptions/urdf/volta/accessories/aruco_marker.urdf.xacro (robot description, xacro)
@@ -27,29 +27,29 @@
 	<xacro:property name="PI" value="3.14159" />
 	<xacro:macro name="aruco_marker" params="frame:=aruco_marker robot_namespace:=/">
-		<link name="${frame}_back_0">
-			<visual>
-				<origin xyz="0 0 0" />
-				<geometry>
-					<mesh filename="package://descriptions/urdf/volta/meshes/${robot_namespace}_aruco.dae" scale="0.3 0.3 0.3"/>
-				</geometry>
-			</visual>
-			<collision>
-				<origin xyz="0 0 0" />
-				<geometry>
-					<mesh filename="package://descriptions/urdf/volta/meshes/${robot_namespace}_aruco.dae" scale="0.3 0.3 0.3"/>
-				</geometry>
-			</collision>
-		</link>
+		<!-- <link name="${frame}_back_0">
+			<visual>
+				<origin xyz="0 0 0" />
+				<geometry>
+					<mesh filename="package://descriptions/urdf/volta/meshes/${robot_namespace}_aruco.dae" scale="0.6 0.6 0.6"/>
+				</geometry>
+			</visual>
+			<collision>
+				<origin xyz="0 0 0" />
+				<geometry>
+					<mesh filename="package://descriptions/urdf/volta/meshes/${robot_namespace}_aruco.dae" scale="0.6 0.6 0.6"/>
+				</geometry>
+			</collision>
+		</link> -->
 		<link name="${frame}_back_1">
 			<visual>
 				<origin xyz="0 0 0" />
 				<geometry>
-					<mesh filename="package://descriptions/urdf/volta/meshes/${robot_namespace}_aruco.dae" scale="0.3 0.3 0.3"/>
-				</geometry>
-			</visual>
-			<collision>
-				<origin xyz="0 0 0" />
-				<geometry>
-					<mesh filename="package://descriptions/urdf/volta/meshes/${robot_namespace}_aruco.dae" scale="0.3 0.3 0.3"/>
+					<mesh filename="package://descriptions/urdf/volta/meshes/${robot_namespace}_aruco.dae" scale="0.6 0.6 0.6"/>
+				</geometry>
+			</visual>
+			<collision>
+				<origin xyz="0 0 0" />
+				<geometry>
+					<mesh filename="package://descriptions/urdf/volta/meshes/${robot_namespace}_aruco.dae" scale="0.6 0.6 0.6"/>
 				</geometry>
 			</collision>
@@ -59,39 +59,39 @@
 				<origin xyz="0 0 0" />
 				<geometry>
-					<mesh filename="package://descriptions/urdf/volta/meshes/${robot_namespace}_aruco.dae" scale="0.3 0.3 0.3"/>
-				</geometry>
-			</visual>
-			<collision>
-				<origin xyz="0 0 0" />
-				<geometry>
-					<mesh filename="package://descriptions/urdf/volta/meshes/${robot_namespace}_aruco.dae" scale="0.3 0.3 0.3"/>
-				</geometry>
-			</collision>
-		</link>
-		<link name="${frame}_front_0">
-			<visual>
-				<origin xyz="0 0 0" />
-				<geometry>
-					<mesh filename="package://descriptions/urdf/volta/meshes/${robot_namespace}_aruco.dae" scale="0.3 0.3 0.3"/>
-				</geometry>
-			</visual>
-			<collision>
-				<origin xyz="0 0 0" />
-				<geometry>
-					<mesh filename="package://descriptions/urdf/volta/meshes/${robot_namespace}_aruco.dae" scale="0.3 0.3 0.3"/>
-				</geometry>
-			</collision>
-		</link>
+					<mesh filename="package://descriptions/urdf/volta/meshes/${robot_namespace}_aruco.dae" scale="0.6 0.6 0.6"/>
+				</geometry>
+			</visual>
+			<collision>
+				<origin xyz="0 0 0" />
+				<geometry>
+					<mesh filename="package://descriptions/urdf/volta/meshes/${robot_namespace}_aruco.dae" scale="0.6 0.6 0.6"/>
+				</geometry>
+			</collision>
+		</link>
+		<!-- <link name="${frame}_front_0">
+			<visual>
+				<origin xyz="0 0 0" />
+				<geometry>
+					<mesh filename="package://descriptions/urdf/volta/meshes/${robot_namespace}_aruco.dae" scale="0.6 0.6 0.6"/>
+				</geometry>
+			</visual>
+			<collision>
+				<origin xyz="0 0 0" />
+				<geometry>
+					<mesh filename="package://descriptions/urdf/volta/meshes/${robot_namespace}_aruco.dae" scale="0.6 0.6 0.6"/>
+				</geometry>
+			</collision>
+		</link> -->
 		<link name="${frame}_front_1">
 			<visual>
 				<origin xyz="0 0 0" />
 				<geometry>
-					<mesh filename="package://descriptions/urdf/volta/meshes/${robot_namespace}_aruco.dae" scale="0.3 0.3 0.3"/>
-				</geometry>
-			</visual>
-			<collision>
-				<origin xyz="0 0 0" />
-				<geometry>
-					<mesh filename="package://descriptions/urdf/volta/meshes/${robot_namespace}_aruco.dae" scale="0.3 0.3 0.3"/>
+					<mesh filename="package://descriptions/urdf/volta/meshes/${robot_namespace}_aruco.dae" scale="0.6 0.6 0.6"/>
+				</geometry>
+			</visual>
+			<collision>
+				<origin xyz="0 0 0" />
+				<geometry>
+					<mesh filename="package://descriptions/urdf/volta/meshes/${robot_namespace}_aruco.dae" scale="0.6 0.6 0.6"/>
 				</geometry>
 			</collision>
@@ -101,39 +101,39 @@
 				<origin xyz="0 0 0" />
 				<geometry>
-					<mesh filename="package://descriptions/urdf/volta/meshes/${robot_namespace}_aruco.dae" scale="0.3 0.3 0.3"/>
-				</geometry>
-			</visual>
-			<collision>
-				<origin xyz="0 0 0" />
-				<geometry>
-					<mesh filename="package://descriptions/urdf/volta/meshes/${robot_namespace}_aruco.dae" scale="0.3 0.3 0.3"/>
-				</geometry>
-			</collision>
-		</link>
-		<link name="${frame}_right_0">
-			<visual>
-				<origin xyz="0 0 0" />
-				<geometry>
-					<mesh filename="package://descriptions/urdf/volta/meshes/${robot_namespace}_aruco.dae" scale="0.3 0.3 0.3"/>
-				</geometry>
-			</visual>
-			<collision>
-				<origin xyz="0 0 0" />
-				<geometry>
-					<mesh filename="package://descriptions/urdf/volta/meshes/${robot_namespace}_aruco.dae" scale="0.3 0.3 0.3"/>
-				</geometry>
-			</collision>
-		</link>
+					<mesh filename="package://descriptions/urdf/volta/meshes/${robot_namespace}_aruco.dae" scale="0.6 0.6 0.6"/>
+				</geometry>
+			</visual>
+			<collision>
+				<origin xyz="0 0 0" />
+				<geometry>
+					<mesh filename="package://descriptions/urdf/volta/meshes/${robot_namespace}_aruco.dae" scale="0.6 0.6 0.6"/>
+				</geometry>
+			</collision>
+		</link>
+		<!-- <link name="${frame}_right_0">
+			<visual>
+				<origin xyz="0 0 0" />
+				<geometry>
+					<mesh filename="package://descriptions/urdf/volta/meshes/${robot_namespace}_aruco.dae" scale="0.6 0.6 0.6"/>
+				</geometry>
+			</visual>
+			<collision>
+				<origin xyz="0 0 0" />
+				<geometry>
+					<mesh filename="package://descriptions/urdf/volta/meshes/${robot_namespace}_aruco.dae" scale="0.6 0.6 0.6"/>
+				</geometry>
+			</collision>
+		</link> -->
 		<link name="${frame}_right_1">
 			<visual>
 				<origin xyz="0 0 0" />
 				<geometry>
-					<mesh filename="package://descriptions/urdf/volta/meshes/${robot_namespace}_aruco.dae" scale="0.3 0.3 0.3"/>
-				</geometry>
-			</visual>
-			<collision>
-				<origin xyz="0 0 0" />
-				<geometry>
-					<mesh filename="package://descriptions/urdf/volta/meshes/${robot_namespace}_aruco.dae" scale="0.3 0.3 0.3"/>
+					<mesh filename="package://descriptions/urdf/volta/meshes/${robot_namespace}_aruco.dae" scale="0.6 0.6 0.6"/>
+				</geometry>
+			</visual>
+			<collision>
+				<origin xyz="0 0 0" />
+				<geometry>
+					<mesh filename="package://descriptions/urdf/volta/meshes/${robot_namespace}_aruco.dae" scale="0.6 0.6 0.6"/>
 				</geometry>
 			</collision>
@@ -143,39 +143,39 @@
 				<origin xyz="0 0 0" />
 				<geometry>
-					<mesh filename="package://descriptions/urdf/volta/meshes/${robot_namespace}_aruco.dae" scale="0.3 0.3 0.3"/>
-				</geometry>
-			</visual>
-			<collision>
-				<origin xyz="0 0 0" />
-				<geometry>
-					<mesh filename="package://descriptions/urdf/volta/meshes/${robot_namespace}_aruco.dae" scale="0.3 0.3 0.3"/>
-				</geometry>
-			</collision>
-		</link>
-		<link name="${frame}_left_0">
-			<visual>
-				<origin xyz="0 0 0" />
-				<geometry>
-					<mesh filename="package://descriptions/urdf/volta/meshes/${robot_namespace}_aruco.dae" scale="0.3 0.3 0.3"/>
-				</geometry>
-			</visual>
-			<collision>
-				<origin xyz="0 0 0" />
-				<geometry>
-					<mesh filename="package://descriptions/urdf/volta/meshes/${robot_namespace}_aruco.dae" scale="0.3 0.3 0.3"/>
-				</geometry>
-			</collision>
-		</link>
+					<mesh filename="package://descriptions/urdf/volta/meshes/${robot_namespace}_aruco.dae" scale="0.6 0.6 0.6"/>
+				</geometry>
+			</visual>
+			<collision>
+				<origin xyz="0 0 0" />
+				<geometry>
+					<mesh filename="package://descriptions/urdf/volta/meshes/${robot_namespace}_aruco.dae" scale="0.6 0.6 0.6"/>
+				</geometry>
+			</collision>
+		</link>
+		<!-- <link name="${frame}_left_0">
+			<visual>
+				<origin xyz="0 0 0" />
+				<geometry>
+					<mesh filename="package://descriptions/urdf/volta/meshes/${robot_namespace}_aruco.dae" scale="0.6 0.6 0.6"/>
+				</geometry>
+			</visual>
+			<collision>
+				<origin xyz="0 0 0" />
+				<geometry>
+					<mesh filename="package://descriptions/urdf/volta/meshes/${robot_namespace}_aruco.dae" scale="0.6 0.6 0.6"/>
+				</geometry>
+			</collision>
+		</link> -->
 		<link name="${frame}_left_1">
 			<visual>
 				<origin xyz="0 0 0" />
 				<geometry>
-					<mesh filename="package://descriptions/urdf/volta/meshes/${robot_namespace}_aruco.dae" scale="0.3 0.3 0.3"/>
-				</geometry>
-			</visual>
-			<collision>
-				<origin xyz="0 0 0" />
-				<geometry>
-					<mesh filename="package://descriptions/urdf/volta/meshes/${robot_namespace}_aruco.dae" scale="0.3 0.3 0.3"/>
+					<mesh filename="package://descriptions/urdf/volta/meshes/${robot_namespace}_aruco.dae" scale="0.6 0.6 0.6"/>
+				</geometry>
+			</visual>
+			<collision>
+				<origin xyz="0 0 0" />
+				<geometry>
+					<mesh filename="package://descriptions/urdf/volta/meshes/${robot_namespace}_aruco.dae" scale="0.6 0.6 0.6"/>
 				</geometry>
 			</collision>
@@ -185,71 +185,71 @@
 				<origin xyz="0 0 0" />
 				<geometry>
-					<mesh filename="package://descriptions/urdf/volta/meshes/${robot_namespace}_aruco.dae" scale="0.3 0.3 0.3"/>
-				</geometry>
-			</visual>
-			<collision>
-				<origin xyz="0 0 0" />
-				<geometry>
-					<mesh filename="package://descriptions/urdf/volta/meshes/${robot_namespace}_aruco.dae" scale="0.3 0.3 0.3"/>
-				</geometry>
-			</collision>
-		</link>
-		<joint name="aruco_marker_joint_back_0" type="fixed">
+					<mesh filename="package://descriptions/urdf/volta/meshes/${robot_namespace}_aruco.dae" scale="0.6 0.6 0.6"/>
+				</geometry>
+			</visual>
+			<collision>
+				<origin xyz="0 0 0" />
+				<geometry>
+					<mesh filename="package://descriptions/urdf/volta/meshes/${robot_namespace}_aruco.dae" scale="0.6 0.6 0.6"/>
+				</geometry>
+			</collision>
+		</link>
+		<!-- <joint name="aruco_marker_joint_back_0" type="fixed">
 			<origin xyz="-0.27 0 0.15" rpy="0 -${PI/2} 0" />
 			<parent link="base_link" />
 			<child link="${frame}_back_0" />
-		</joint>
+		</joint> -->
 		<joint name="aruco_marker_joint_back_1" type="fixed">
-			<origin xyz="-0.27 -0.125 0.15" rpy="0 -${PI/2} 0" />
+			<origin xyz="-0.27 -0.12 0.1" rpy="0 -${PI/2} 0" />
 			<parent link="base_link" />
 			<child link="${frame}_back_1" />
 		</joint>
 		<joint name="aruco_marker_joint_back_2" type="fixed">
-			<origin xyz="-0.27 0.125 0.15" rpy="0 -${PI/2} 0" />
+			<origin xyz="-0.27 0.12 0.1" rpy="0 -${PI/2} 0" />
 			<parent link="base_link" />
 			<child link="${frame}_back_2" />
 		</joint>
-		<joint name="aruco_marker_joint_front_0" type="fixed">
+		<!-- <joint name="aruco_marker_joint_front_0" type="fixed">
 			<origin xyz="0.27 0 0.15" rpy="0 ${PI/2} 0" />
 			<parent link="base_link" />
 			<child link="${frame}_front_0" />
-		</joint>
+		</joint> -->
 		<joint name="aruco_marker_joint_front_1" type="fixed">
-			<origin xyz="0.27 -0.125 0.15" rpy="0 ${PI/2} 0" />
+			<origin xyz="0.27 -0.12 0.1" rpy="0 ${PI/2} 0" />
 			<parent link="base_link" />
 			<child link="${frame}_front_1" />
 		</joint>
 		<joint name="aruco_marker_joint_front_2" type="fixed">
-			<origin xyz="0.27 0.125 0.15" rpy="0 ${PI/2} 0" />
+			<origin xyz="0.27 0.12 0.1" rpy="0 ${PI/2} 0" />
 			<parent link="base_link" />
 			<child link="${frame}_front_2" />
 		</joint>
-		<joint name="aruco_marker_joint_right_0" type="fixed">
+		<!-- <joint name="aruco_marker_joint_right_0" type="fixed">
 			<origin xyz="0 -0.2 0.15" rpy="${PI/2} 0 0" />
 			<parent link="base_link" />
 			<child link="${frame}_right_0" />
-		</joint>
+		</joint> -->
 		<joint name="aruco_marker_joint_right_1" type="fixed">
-			<origin xyz="-0.2 -0.2 0.15" rpy="${PI/2} 0 0" />
+			<origin xyz="-0.1 -0.2 0.1" rpy="${PI/2} 0 0" />
 			<parent link="base_link" />
 			<child link="${frame}_right_1" />
 		</joint>
 		<joint name="aruco_marker_joint_right_2" type="fixed">
-			<origin xyz="0.2 -0.2 0.15" rpy="${PI/2} 0 0" />
+			<origin xyz="0.1 -0.2 0.1" rpy="${PI/2} 0 0" />
 			<parent link="base_link" />
 			<child link="${frame}_right_2" />
 		</joint>
-		<joint name="aruco_marker_joint_left_0" type="fixed">
+		<!-- <joint name="aruco_marker_joint_left_0" type="fixed">
 			<origin xyz="0 0.2 0.15" rpy="-${PI/2} 0 0" />
 			<parent link="base_link" />
 			<child link="${frame}_left_0" />
-		</joint>
+		</joint> -->
 		<joint name="aruco_marker_joint_left_1" type="fixed">
-			<origin xyz="-0.2 0.2 0.15" rpy="-${PI/2} 0 0" />
+			<origin xyz="-0.1 0.2 0.1" rpy="-${PI/2} 0 0" />
 			<parent link="base_link" />
 			<child link="${frame}_left_1" />
 		</joint>
 		<joint name="aruco_marker_joint_left_2" type="fixed">
-			<origin xyz="0.2 0.2 0.15" rpy="-${PI/2} 0 0" />
+			<origin xyz="0.1 0.2 0.1" rpy="-${PI/2} 0 0" />
 			<parent link="base_link" />
 			<child link="${frame}_left_2" />

File: descriptions/urdf/volta/accessories/camera_volta.urdf.xacro (robot description, xacro)
@@ -89,15 +89,15 @@
             <parent link="base_link"/>
             <child link="${frame}_front"/>
-            <origin xyz="${camera_joint_x} ${camera_joint_y} ${camera_joint_z + 0.0125}"/>
+            <origin xyz="${camera_joint_x + 0.05} ${camera_joint_y} ${camera_joint_z + 0.0225}"/>
         </joint>
         <joint name="base_to_camera_right" type="fixed">
             <parent link="base_link"/>
             <child link="${frame}_right"/>
-            <origin xyz="0.0 -0.2 ${camera_joint_z + 0.0125}" rpy="0 0 -1.5707"/>
+            <origin xyz="0.0 -0.2 ${camera_joint_z + 0.0225}" rpy="0 0 -1.5707"/>
         </joint>
         <joint name="base_to_camera_left" type="fixed">
             <parent link="base_link"/>
             <child link="${frame}_left"/>
-            <origin xyz="0.0 0.2 ${camera_joint_z + 0.0125}" rpy="0 0 1.5707"/>
+            <origin xyz="0.0 0.2 ${camera_joint_z + 0.0225}" rpy="0 0 1.5707"/>
         </joint>
         </xacro:if>
